Commit message: Apply new scaling to test robot

File: data/robots/test_robot/my_robot.urdf (robot description, URDF)
Before this commit: robot origins, 3 links, 2 joints
Links:
- link ltorso: geometry visual mesh filename=Armar4.dae scale=1000 1000 1000
- link mtorso: geometry visual mesh filename=MMM.dae scale=1500 1500 1500
- link utorso: geometry visual mesh filename=MMM.dae scale=1500 1500 1500
