Commit message: fix armar4 urdf model and eefs add load modes to urdf import (structure, collisionmodel, full) add urdf-eef load tests

File: data/robots/Armar4/urdf/Armar4.urdf (robot description, URDF)
Before this commit: robot Armar4, 80 links, 79 joints
Links:
- removed link ArmL_Elb1_joint_link
- removed link ArmL_Elb2_joint_link
- removed link ArmL_Sho1_joint_link
- removed link ArmL_Sho2_joint_link
- removed link ArmL_Sho3_joint_link
- removed link ArmL_Sho4_joint_link
- removed link ArmL_Wri1_joint_link
- removed link ArmL_Wri2_joint_link
- removed link ArmR_Elb1_joint_link
- removed link ArmR_Elb2_joint_link
- removed link ArmR_Sho1_joint_link
- removed link ArmR_Sho2_joint_link
- removed link ArmR_Sho3_joint_link
- removed link ArmR_Sho4_joint_link
- removed link ArmR_Wri1_joint_link
- removed link ArmR_Wri2_joint_link
- removed link EyeL_1_joint_link
- removed link EyeL_2_joint_link
- removed link EyeR_1_joint_link
- removed link EyeR_2_joint_link
- removed link HandL_Finger_Index1_joint_link
- removed link HandL_Finger_Index2_joint_link
- removed link HandL_Finger_Middle1_joint_link
- removed link HandL_Finger_Middle2_joint_link
- removed link HandL_Finger_Pinky1_joint_link
- removed link HandL_Finger_Pinky2_joint_link
- removed link HandL_Finger_Ring1_joint_link
- removed link HandL_Finger_Ring2_joint_link
- removed link HandL_Finger_Thumb1_joint_link
- removed link HandL_Finger_Thumb2_joint_link
- removed link HandL_Finger_Thumb3_joint_link
- removed link HandR_Finger_Index1_joint_link
- removed link HandR_Finger_Index2_joint_link
- removed link HandR_Finger_Middle1_joint_link
- removed link HandR_Finger_Middle2_joint_link
- removed link HandR_Finger_Ring1_joint_link
- removed link HandR_Finger_Ring2_joint_link
- removed link HandR_Finger_Small1_joint_link
- removed link HandR_Finger_Small2_joint_link
- removed link HandR_Finger_Thumb1_joint_link
- removed link HandR_Finger_Thumb2_joint_link
- removed link HandR_Finger_Thumb3_joint_link
- removed link Head_1_joint_link
- removed link Head_2_joint_link
- removed link LegL_Ank1_joint_link
- removed link LegL_Ank2_joint_link
- removed link LegL_Heel_joint_link
- removed link LegL_Hip1_joint_link
- removed link LegL_Hip2_joint_link
- removed link LegL_Hip3_joint_link
- removed link LegL_Knee_joint_link
- removed link LegL_Toe2_joint_link
- removed link LegL_Toe_joint_link
- removed link LegR_Ank1_joint_link
- removed link LegR_Ank2_joint_link
- removed link LegR_Heel_joint_link
- removed link LegR_Hip1_joint_link
- removed link LegR_Hip2_joint_link
- removed link LegR_Hip3_joint_link
- removed link LegR_Knee_joint_link
- removed link LegR_Toe2_joint_link
- removed link LegR_Toe_joint_link
- removed link Neck_1_joint_link
- removed link Neck_2_joint_link
- removed link Neck_3_joint_link
- removed link Root_joint_link
- removed link Torso_Pitch_joint_link
- removed link Torso_Yaw_joint_link
- added link ArmL_Elb1_link, mass 0.61; collision mesh filename=stl/ArmL_Elb1_joint_col.stl scale=1 1 1; visual mesh filename=stl/ArmL_Elb1_joint_visu.stl scale=1 1 1
- added link ArmL_Elb2_link, mass 0.43; collision mesh filename=stl/ArmL_Elb2_joint_col.stl scale=1 1 1; visual mesh filename=stl/ArmL_Elb2_joint_visu.stl scale=1 1 1
- added link ArmL_Sho1_link, mass 0.58; collision mesh filename=stl/ArmL_Sho1_joint_col.stl scale=1 1 1; visual mesh filename=stl/ArmL_Sho1_joint_visu.stl scale=1 1 1
- added link ArmL_Sho2_link, mass 0.52; collision mesh filename=stl/ArmL_Sho2_joint_col.stl scale=1 1 1; visual mesh filename=stl/ArmL_Sho2_joint_visu.stl scale=1 1 1
- added link ArmL_Sho3_link, mass 0.51; collision mesh filename=stl/ArmL_Sho3_joint_col.stl scale=1 1 1; visual mesh filename=stl/ArmL_Sho3_joint_visu.stl scale=1 1 1
- added link ArmL_Sho4_link, mass 1.44; collision mesh filename=stl/ArmL_Sho4_joint_col.stl scale=1 1 1; visual mesh filename=stl/ArmL_Sho4_joint_visu.stl scale=1 1 1
- added link ArmL_Wri1_link, mass 0.5; collision mesh filename=stl/sphere10.stl scale=1 1 1; visual mesh filename=stl/ArmL_Wri1_joint_visu.stl scale=1 1 1
- added link ArmL_Wri2_link, mass 0.58; collision mesh filename=stl/ArmL_Wri2_joint_col.stl scale=1 1 1; visual mesh filename=stl/ArmL_Wri2_joint_visu.stl scale=1 1 1
- added link ArmR_Elb1_link, mass 0.61; collision mesh filename=stl/ArmR_Elb1_joint_col.stl scale=1 1 1; visual mesh filename=stl/ArmR_Elb1_joint_visu.stl scale=1 1 1
- added link ArmR_Elb2_link, mass 0.43; collision mesh filename=stl/ArmR_Elb2_joint_col.stl scale=1 1 1; visual mesh filename=stl/ArmR_Elb2_joint_visu.stl scale=1 1 1
- added link ArmR_Sho1_link, mass 0.77; collision mesh filename=stl/ArmR_Sho1_joint_col.stl scale=1 1 1; visual mesh filename=stl/ArmR_Sho1_joint_visu.stl scale=1 1 1
- added link ArmR_Sho2_link, mass 0.58; collision mesh filename=stl/ArmR_Sho2_joint_col.stl scale=1 1 1; visual mesh filename=stl/ArmR_Sho2_joint_visu.stl scale=1 1 1
- added link ArmR_Sho3_link, mass 0.51; collision mesh filename=stl/ArmR_Sho3_joint_col.stl scale=1 1 1; visual mesh filename=stl/ArmR_Sho3_joint_visu.stl scale=1 1 1
- added link ArmR_Sho4_link, mass 1.44; collision mesh filename=stl/ArmR_Sho4_joint_col.stl scale=1 1 1; visual mesh filename=stl/ArmR_Sho4_joint_visu.stl scale=1 1 1
- added link ArmR_Wri1_link, mass 0.5; collision mesh filename=stl/sphere10.stl scale=1 1 1; visual mesh filename=stl/ArmR_Wri1_joint_visu.stl scale=1 1 1
- added link ArmR_Wri2_link, mass 0.58; collision mesh filename=stl/ArmR_Wri2_joint_col.stl scale=1 1 1; visual mesh filename=stl/ArmR_Wri2_joint_visu.stl scale=1 1 1
- added link EyeL_1_link, mass 0.05; collision mesh filename=stl/EyeL_1_joint_visu.stl scale=1 1 1; visual mesh filename=stl/EyeL_1_joint_visu.stl scale=1 1 1
- added link EyeL_2_link, mass 0.05; collision mesh filename=stl/EyeL_2_joint_col.stl scale=1 1 1; visual mesh filename=stl/EyeL_2_joint_visu.stl scale=1 1 1
- added link EyeR_1_link, mass 0.05; collision mesh filename=stl/EyeR_1_joint_visu.stl scale=1 1 1; visual mesh filename=stl/EyeR_1_joint_visu.stl scale=1 1 1
- added link EyeR_2_link, mass 0.05; collision mesh filename=stl/EyeR_2_joint_visu.stl scale=1 1 1; visual mesh filename=stl/EyeR_2_joint_visu.stl scale=1 1 1
- added link HandL_Finger_Index1_link, mass 0.05; collision mesh filename=stl/HandL_Finger_Index1_joint_col.stl scale=1 1 1; visual mesh filename=stl/HandL_Finger_Index1_joint_visu.stl scale=1 1 1
- added link HandL_Finger_Index2_link, mass 0.05; collision mesh filename=stl/HandL_Finger_Index2_joint_col.stl scale=1 1 1; visual mesh filename=stl/HandL_Finger_Index2_joint_visu.stl scale=1 1 1
- added link HandL_Finger_Middle1_link, mass 0.05; collision mesh filename=stl/HandL_Finger_Middle1_joint_col.stl scale=1 1 1; visual mesh filename=stl/HandL_Finger_Middle1_joint_visu.stl scale=1 1 1
- added link HandL_Finger_Middle2_link, mass 0.05; collision mesh filename=stl/HandL_Finger_Middle2_joint_col.stl scale=1 1 1; visual mesh filename=stl/HandL_Finger_Middle2_joint_visu.stl scale=1 1 1
- added link HandL_Finger_Pinky1_link, mass 0.05; collision mesh filename=stl/HandL_Finger_Pinky1_joint_col.stl scale=1 1 1; visual mesh filename=stl/HandL_Finger_Pinky1_joint_visu.stl scale=1 1 1
- added link HandL_Finger_Pinky2_link, mass 0.05; collision mesh filename=stl/HandL_Finger_Pinky2_joint_col.stl scale=1 1 1; visual mesh filename=stl/HandL_Finger_Pinky2_joint_visu.stl scale=1 1 1
- added link HandL_Finger_Ring1_link, mass 0.05; collision mesh filename=stl/HandL_Finger_Ring1_joint_col.stl scale=1 1 1; visual mesh filename=stl/HandL_Finger_Ring1_joint_visu.stl scale=1 1 1
- added link HandL_Finger_Ring2_link, mass 0.05; collision mesh filename=stl/HandL_Finger_Ring2_joint_col.stl scale=1 1 1; visual mesh filename=stl/HandL_Finger_Ring2_joint_visu.stl scale=1 1 1
- added link HandL_Finger_Thumb1_link, mass 0.05; collision mesh filename=stl/HandL_Finger_Thumb1_joint_col.stl scale=1 1 1; visual mesh filename=stl/HandL_Finger_Thumb1_joint_visu.stl scale=1 1 1
- added link HandL_Finger_Thumb2_link, mass 0.05; collision mesh filename=stl/HandL_Finger_Thumb2_joint_col.stl scale=1 1 1; visual mesh filename=stl/HandL_Finger_Thumb2_joint_visu.stl scale=1 1 1
- added link HandL_Finger_Thumb3_link, mass 0.05; collision mesh filename=stl/HandL_Finger_Thumb3_joint_col.stl scale=1 1 1; visual mesh filename=stl/HandL_Finger_Thumb3_joint_visu.stl scale=1 1 1
- added link HandR_Finger_Index1_link, mass 0.05; collision mesh filename=stl/HandR_Finger_Index1_joint_col.stl scale=1 1 1; visual mesh filename=stl/HandR_Finger_Index1_joint_visu.stl scale=1 1 1
- added link HandR_Finger_Index2_link, mass 0.05; collision mesh filename=stl/HandR_Finger_Index2_joint_col.stl scale=1 1 1; visual mesh filename=stl/HandR_Finger_Index2_joint_visu.stl scale=1 1 1
- added link HandR_Finger_Middle1_link, mass 0.05; collision mesh filename=stl/HandR_Finger_Middle1_joint_col.stl scale=1 1 1; visual mesh filename=stl/HandR_Finger_Middle1_joint_visu.stl scale=1 1 1
- added link HandR_Finger_Middle2_link, mass 0.05; collision mesh filename=stl/HandR_Finger_Middle2_joint_col.stl scale=1 1 1; visual mesh filename=stl/HandR_Finger_Middle2_joint_visu.stl scale=1 1 1
- added link HandR_Finger_Pinky1_link, mass 0.05; collision mesh filename=stl/HandR_Finger_Pinky1_joint_col.stl scale=1 1 1; visual mesh filename=stl/HandR_Finger_Pinky1_joint_visu.stl scale=1 1 1
- added link HandR_Finger_Pinky2_link, mass 0.05; collision mesh filename=stl/HandR_Finger_Pinky2_joint_col.stl scale=1 1 1; visual mesh filename=stl/HandR_Finger_Pinky2_joint_visu.stl scale=1 1 1
- added link HandR_Finger_Ring1_link, mass 0.05; collision mesh filename=stl/HandR_Finger_Ring1_joint_col.stl scale=1 1 1; visual mesh filename=stl/HandR_Finger_Ring1_joint_visu.stl scale=1 1 1
- added link HandR_Finger_Ring2_link, mass 0.05; collision mesh filename=stl/HandR_Finger_Ring2_joint_col.stl scale=1 1 1; visual mesh filename=stl/HandR_Finger_Ring2_joint_visu.stl scale=1 1 1
- added link HandR_Finger_Thumb1_link, mass 0.05; collision mesh filename=stl/HandR_Finger_Thumb1_joint_col.stl scale=1 1 1; visual mesh filename=stl/HandR_Finger_Thumb1_joint_visu.stl scale=1 1 1
- added link HandR_Finger_Thumb2_link, mass 0.05; collision mesh filename=stl/HandR_Finger_Thumb2_joint_col.stl scale=1 1 1; visual mesh filename=stl/HandR_Finger_Thumb2_joint_visu.stl scale=1 1 1
- added link HandR_Finger_Thumb3_link, mass 0.05; collision mesh filename=stl/HandR_Finger_Thumb3_joint_col.stl scale=1 1 1; visual mesh filename=stl/HandR_Finger_Thumb3_joint_visu.stl scale=1 1 1
- added link Head_1_link, mass 0.07; collision mesh filename=stl/Head_1_joint_col.stl scale=1 1 1; visual mesh filename=stl/Head_1_joint_visu.stl scale=1 1 1
- added link Head_2_link, mass 1.34; collision mesh filename=stl/Head_2_joint_col.stl scale=1 1 1; visual mesh filename=stl/Head_2_joint_visu.stl scale=1 1 1
- added link LegL_Ank1_link, mass 0.5; collision mesh filename=stl/sphere10.stl scale=1 1 1
- added link LegL_Ank2_link, mass 0
- added link LegL_Heel_link, mass 0.05; collision mesh filename=stl/LegL_Heel_joint_visu.stl scale=1 1 1; visual mesh filename=stl/LegL_Heel_joint_visu.stl scale=1 1 1
- added link LegL_Hip1_link, mass 1.33; collision mesh filename=stl/LegL_Hip1_joint_col.stl scale=1 1 1; visual mesh filename=stl/LegL_Hip1_joint_visu.stl scale=1 1 1
- added link LegL_Hip2_link, mass 0.36; collision mesh filename=stl/LegL_Hip2_joint_col.stl scale=1 1 1; visual mesh filename=stl/LegL_Hip2_joint_visu.stl scale=1 1 1
- added link LegL_Hip3_link, mass 5.06; collision mesh filename=stl/LegL_Hip3_joint_col.stl scale=1 1 1; visual mesh filename=stl/LegL_Hip3_joint_visu.stl scale=1 1 1
- added link LegL_Knee_link, mass 4.25; collision mesh filename=stl/LegL_Knee_joint_col.stl scale=1 1 1; visual mesh filename=stl/LegL_Knee_joint_visu.stl scale=1 1 1
- added link LegL_Toe2_link, mass 0.13; collision mesh filename=stl/LegL_Toe2_joint_visu.stl scale=1 1 1; visual mesh filename=stl/LegL_Toe2_joint_visu.stl scale=1 1 1
- added link LegL_Toe_link, mass 0.1; collision mesh filename=stl/LegL_Toe_joint_visu.stl scale=1 1 1; visual mesh filename=stl/LegL_Toe_joint_visu.stl scale=1 1 1
- added link LegR_Ank1_link, mass 0.5; collision mesh filename=stl/sphere10.stl scale=1 1 1
- added link LegR_Ank2_link, mass 0
- added link LegR_Heel_link, mass 0.05; collision mesh filename=stl/LegR_Heel_joint_visu.stl scale=1 1 1; visual mesh filename=stl/LegR_Heel_joint_visu.stl scale=1 1 1
- added link LegR_Hip1_link, mass 1.33; collision mesh filename=stl/LegR_Hip1_joint_col.stl scale=1 1 1; visual mesh filename=stl/LegR_Hip1_joint_visu.stl scale=1 1 1
- added link LegR_Hip2_link, mass 0.36; collision mesh filename=stl/LegR_Hip2_joint_col.stl scale=1 1 1; visual mesh filename=stl/LegR_Hip2_joint_visu.stl scale=1 1 1
- added link LegR_Hip3_link, mass 5.06; collision mesh filename=stl/LegR_Hip3_joint_col.stl scale=1 1 1; visual mesh filename=stl/LegR_Hip3_joint_visu.stl scale=1 1 1
- added link LegR_Knee_link, mass 4.25; collision mesh filename=stl/LegR_Knee_joint_col.stl scale=1 1 1; visual mesh filename=stl/LegR_Knee_joint_visu.stl scale=1 1 1
- added link LegR_Toe2_link, mass 0.13; collision mesh filename=stl/LegR_Toe2_joint_visu.stl scale=1 1 1; visual mesh filename=stl/LegR_Toe2_joint_visu.stl scale=1 1 1
- added link LegR_Toe_link, mass 0.1; collision mesh filename=stl/LegR_Toe_joint_visu.stl scale=1 1 1; visual mesh filename=stl/LegR_Toe_joint_visu.stl scale=1 1 1
- added link Neck_1_link, mass 0.14; collision mesh filename=stl/Neck_1_joint_col.stl scale=1 1 1; visual mesh filename=stl/Neck_1_joint_visu.stl scale=1 1 1
- added link Neck_2_link, mass 0.13; collision mesh filename=stl/Neck_2_joint_col.stl scale=1 1 1; visual mesh filename=stl/Neck_2_joint_visu.stl scale=1 1 1
- added link Neck_3_link, mass 0.25; collision mesh filename=stl/Neck_3_joint_col.stl scale=1 1 1; visual mesh filename=stl/Neck_3_joint_visu.stl scale=1 1 1
- added link Root_link, mass 5; collision mesh filename=stl/Root_joint_col.stl scale=1 1 1; visual mesh filename=stl/Root_joint_visu.stl scale=1 1 1
- added link Torso_Pitch_link, mass 25.49; collision mesh filename=stl/Torso_Pitch_joint_col.stl scale=1 1 1; visual mesh filename=stl/Torso_Pitch_joint_visu.stl scale=1 1 1
- added link Torso_Yaw_link, mass 5.01; collision mesh filename=stl/Torso_Yaw_joint_col.stl scale=1 1 1; visual mesh filename=stl/Torso_Yaw_joint_visu.stl scale=1 1 1
Joints:
- removed joint ArmL_Elb1_joint_joint
- removed joint ArmL_Elb2_joint_joint
- removed joint ArmL_Sho1_joint_joint
- removed joint ArmL_Sho2_joint_joint
- removed joint ArmL_Sho3_joint_joint
- removed joint ArmL_Sho4_joint_joint
- removed joint ArmL_Wri1_joint_joint
- removed joint ArmL_Wri2_joint_joint
- removed joint ArmR_Elb1_joint_joint
- removed joint ArmR_Elb2_joint_joint
- removed joint ArmR_Sho1_joint_joint
- removed joint ArmR_Sho2_joint_joint
- removed joint ArmR_Sho3_joint_joint
- removed joint ArmR_Sho4_joint_joint
- removed joint ArmR_Wri1_joint_joint
- removed joint ArmR_Wri2_joint_joint
- removed joint EyeL_1_joint_joint
- removed joint EyeL_2_joint_joint
- removed joint EyeR_1_joint_joint
- removed joint EyeR_2_joint_joint
- removed joint HandL_Finger_Index1_joint_joint
- removed joint HandL_Finger_Index2_joint_joint
- removed joint HandL_Finger_Middle1_joint_joint
- removed joint HandL_Finger_Middle2_joint_joint
- removed joint HandL_Finger_Pinky1_joint_joint
- removed joint HandL_Finger_Pinky2_joint_joint
- removed joint HandL_Finger_Ring1_joint_joint
- removed joint HandL_Finger_Ring2_joint_joint
- removed joint HandL_Finger_Thumb1_joint_joint
- removed joint HandL_Finger_Thumb2_joint_joint
- removed joint HandL_Finger_Thumb3_joint_joint
- removed joint HandR_Finger_Index1_joint_joint
- removed joint HandR_Finger_Index2_joint_joint
- removed joint HandR_Finger_Middle1_joint_joint
- removed joint HandR_Finger_Middle2_joint_joint
- removed joint HandR_Finger_Ring1_joint_joint
- removed joint HandR_Finger_Ring2_joint_joint
- removed joint HandR_Finger_Small1_joint_joint
- removed joint HandR_Finger_Small2_joint_joint
- removed joint HandR_Finger_Thumb1_joint_joint
- removed joint HandR_Finger_Thumb2_joint_joint
- removed joint HandR_Finger_Thumb3_joint_joint
- removed joint Head_1_joint_joint
- removed joint Head_2_joint_joint
- removed joint LegL_Ank1_joint_joint
- removed joint LegL_Ank2_joint_joint
- removed joint LegL_Heel_joint_joint
- removed joint LegL_Hip1_joint_joint
- removed joint LegL_Hip2_joint_joint
- removed joint LegL_Hip3_joint_joint
- removed joint LegL_Knee_joint_joint
- removed joint LegL_Toe2_joint_joint
- removed joint LegL_Toe_joint_joint
- removed joint LegR_Ank1_joint_joint
- removed joint LegR_Ank2_joint_joint
- removed joint LegR_Heel_joint_joint
- removed joint LegR_Hip1_joint_joint
- removed joint LegR_Hip2_joint_joint
- removed joint LegR_Hip3_joint_joint
- removed joint LegR_Knee_joint_joint
- removed joint LegR_Toe2_joint_joint
- removed joint LegR_Toe_joint_joint
- removed joint Neck_1_joint_joint
- removed joint Neck_2_joint_joint
- removed joint Neck_3_joint_joint
- removed joint Root_joint_joint
- removed joint Torso_Pitch_joint_joint
- removed joint Torso_Yaw_joint_joint
- added joint ArmL_Elb1_joint: type revolute, parent ArmL_Sho4_link, child ArmL_Elb1_link, origin xyz=-0.0215 -0.01 -0.1974 rpy=1.57079625 -8.74227979e-08 -1.57079625, axis 0 0 1, limit lower=-0.0872665 upper=1.81514 effort=-1 velocity=-1
- added joint ArmL_Elb2_joint: type revolute, parent ArmL_Elb1_link, child ArmL_Elb2_link, origin xyz=0 -0.0858 -0.0205 rpy=-1.57079637 1.57079625 0, axis 0 0 1, limit lower=-3.14159 upper=1.5708 effort=-1 velocity=-1
- added joint ArmL_Sho1_joint: type revolute, parent Torso_Pitch_link, child ArmL_Sho1_link, origin xyz=0 0.2103 0 rpy=1.57079625 -8.74227979e-08 8.74227979e-08, axis 0 0 1, limit lower=0 upper=0.785398 effort=-1 velocity=-1
- added joint ArmL_Sho2_joint: type revolute, parent ArmL_Sho1_link, child ArmL_Sho2_link, origin xyz=0 0.136249 -0.0599 rpy=1.30899704 -8.74227979e-08 8.74227979e-08, axis 0 0 1, limit lower=-0.523599 upper=2.61799 effort=-1 velocity=-1
- added joint ArmL_Sho3_joint: type revolute, parent ArmL_Sho2_link, child ArmL_Sho3_link, origin xyz=0.0165 0 -0.066 rpy=-1.57079637 1.48352981 1.57079637, axis 0 0 1, limit lower=-0.261799 upper=1.39626 effort=-1 velocity=-1
- added joint ArmL_Sho4_joint: type revolute, parent ArmL_Sho3_link, child ArmL_Sho4_link, origin xyz=0 -0.1026 0.0165 rpy=-1.57079637 -0 0, axis 0 0 1, limit lower=-1.39626 upper=2.96706 effort=-1 velocity=-1
- added joint ArmL_Wri1_joint: type revolute, parent ArmL_Elb2_link, child ArmL_Wri1_link, origin xyz=0 0 -0.1642 rpy=-1.57079625 -8.74227979e-08 1.57079625, axis 0 0 1, limit lower=-0.349066 upper=0.349066 effort=-1 velocity=-1
- added joint ArmL_Wri2_joint: type revolute, parent ArmL_Wri1_link, child ArmL_Wri2_link, origin xyz=0 0 0 rpy=1.57079625 -8.74227979e-08 1.57079625, axis 0 0 1, limit lower=-1.5708 upper=1.5708 effort=-1 velocity=-1
- added joint ArmR_Elb1_joint: type revolute, parent ArmR_Sho4_link, child ArmR_Elb1_link, origin xyz=-0.0215 0.01 0.1974 rpy=-1.57079637 -0 1.57079637, axis 0 0 1, limit lower=-0.0872665 upper=1.81514 effort=-1 velocity=-1
- added joint ArmR_Elb2_joint: type revolute, parent ArmR_Elb1_link, child ArmR_Elb2_link, origin xyz=0 -0.0858 -0.0205 rpy=1.57079637 1.57079625 0, axis 0 0 1, limit lower=-3.14159 upper=1.5708 effort=-1 velocity=-1
- added joint ArmR_Sho1_joint: type revolute, parent Torso_Pitch_link, child ArmR_Sho1_link, origin xyz=0 0.2103 0 rpy=-1.57079637 -0 0, axis 0 0 1, limit lower=0 upper=0.785398 effort=-1 velocity=-1
- added joint ArmR_Sho2_joint: type revolute, parent ArmR_Sho1_link, child ArmR_Sho2_link, origin xyz=0 0.136249 0.0599 rpy=-1.30899704 -8.74227979e-08 8.74227979e-08, axis 0 0 1, limit lower=-0.523599 upper=2.61799 effort=-1 velocity=-1
- added joint ArmR_Sho3_joint: type revolute, parent ArmR_Sho2_link, child ArmR_Sho3_link, origin xyz=-0.0165 0 0.066 rpy=-1.57079637 1.48352981 -1.57079637, axis 0 0 1, limit lower=-0.261799 upper=1.39626 effort=-1 velocity=-1
- added joint ArmR_Sho4_joint: type revolute, parent ArmR_Sho3_link, child ArmR_Sho4_link, origin xyz=0 0.1026 0.0165 rpy=-1.57079637 -0 0, axis 0 0 1, limit lower=-1.39626 upper=2.96706 effort=-1 velocity=-1
- added joint ArmR_Wri1_joint: type revolute, parent ArmR_Elb2_link, child ArmR_Wri1_link, origin xyz=-0.0005 0 0.1642 rpy=1.57079637 -0 -1.57079637, axis 0 0 1, limit lower=-0.349066 upper=0.349066 effort=-1 velocity=-1
- added joint ArmR_Wri2_joint: type revolute, parent ArmR_Wri1_link, child ArmR_Wri2_link, origin xyz=0 0 0 rpy=-1.57079637 -0 1.57079637, axis 0 0 1, limit lower=-1.5708 upper=1.5708 effort=-1 velocity=-1
- added joint EyeL_1_joint: type revolute, parent Head_2_link, child EyeL_1_link, origin xyz=-0.0105 0.0726517 -0.06315 rpy=1.57079637 -0 -1.57079637, axis 0 0 1, limit lower=-0.349066 upper=0.349066 effort=-1 velocity=-1
- added joint EyeL_2_joint: type revolute, parent EyeL_1_link, child EyeL_2_link, origin xyz=0 0 0.036 rpy=1.57079637 -0 -1.57079637, axis 0 0 1, limit lower=-0.698132 upper=0.698132 effort=-1 velocity=-1
- added joint EyeR_1_joint: type revolute, parent Head_2_link, child EyeR_1_link, origin xyz=0.015 0.0726517 -0.06315 rpy=1.57079637 -0 -1.57079637, axis 0 0 1, limit lower=-0.349066 upper=0.349066 effort=-1 velocity=-1
- added joint EyeR_2_joint: type revolute, parent EyeR_1_link, child EyeR_2_link, origin xyz=0 0 -0.0315 rpy=-1.57079637 -0 -1.57079637, axis 0 0 1, limit lower=-0.698132 upper=0.698132 effort=-1 velocity=-1
- added joint HandL_Finger_Index1_joint: type revolute, parent ArmL_Wri2_link, child HandL_Finger_Index1_link, origin xyz=0.08965 0.0096 -0.025 rpy=0 0.087266393 0, axis 0 0 1, limit lower=0 upper=1.5708 effort=-1 velocity=-1
- added joint HandL_Finger_Index2_joint: type revolute, parent HandL_Finger_Index1_link, child HandL_Finger_Index2_link, origin xyz=0.0453 -0.0002 0 rpy=0 -0 0, axis 0 0 1, limit lower=0 upper=1.5708 effort=-1 velocity=-1
- added joint HandL_Finger_Middle1_joint: type revolute, parent ArmL_Wri2_link, child HandL_Finger_Middle1_link, origin xyz=0.0913 0.0098 -0.0047 rpy=0 -0 0, axis 0 0 1, limit lower=0 upper=1.5708 effort=-1 velocity=-1
- added joint HandL_Finger_Middle2_joint: type revolute, parent HandL_Finger_Middle1_link, child HandL_Finger_Middle2_link, origin xyz=0.045 -0.00305 0 rpy=0 -0 0, axis 0 0 1, limit lower=0 upper=1.5708 effort=-1 velocity=-1
- added joint HandL_Finger_Pinky1_joint: type revolute, parent ArmL_Wri2_link, child HandL_Finger_Pinky1_link, origin xyz=0.08845 0.0097 0.0317 rpy=0 -0.174532697 0, axis 0 0 1, limit lower=0 upper=1.5708 effort=-1 velocity=-1
- added joint HandL_Finger_Pinky2_joint: type revolute, parent HandL_Finger_Pinky1_link, child HandL_Finger_Pinky2_link, origin xyz=0.027 0 0 rpy=0 -0 0, axis 0 0 1, limit lower=0 upper=1.5708 effort=-1 velocity=-1
- added joint HandL_Finger_Ring1_joint: type revolute, parent ArmL_Wri2_link, child HandL_Finger_Ring1_link, origin xyz=0.0912 0.0098 0.0142 rpy=0 -0.087266393 0, axis 0 0 1, limit lower=0 upper=1.5708 effort=-1 velocity=-1
- added joint HandL_Finger_Ring2_joint: type revolute, parent HandL_Finger_Ring1_link, child HandL_Finger_Ring2_link, origin xyz=0.04 0 0 rpy=0 -0 0, axis 0 0 1, limit lower=0 upper=1.5708 effort=-1 velocity=-1
- added joint HandL_Finger_Thumb1_joint: type revolute, parent ArmL_Wri2_link, child HandL_Finger_Thumb1_link, origin xyz=0.0353 0.0098 -0.0111 rpy=-1.57079637 -0 -1.57079637, axis 0 0 1, limit lower=0 upper=1.5708 effort=-1 velocity=-1
- added joint HandL_Finger_Thumb2_joint: type revolute, parent HandL_Finger_Thumb1_link, child HandL_Finger_Thumb2_link, origin xyz=0.0035 0.03 0.0043 rpy=0 1.57079625 0, axis 0 0 1, limit lower=0 upper=1.5708 effort=-1 velocity=-1
- added joint HandL_Finger_Thumb3_joint: type revolute, parent HandL_Finger_Thumb2_link, child HandL_Finger_Thumb3_link, origin xyz=0.0029 0.0294 0 rpy=0 -0 0, axis 0 0 1, limit lower=0 upper=1.5708 effort=-1 velocity=-1
- added joint HandR_Finger_Index1_joint: type revolute, parent ArmR_Wri2_link, child HandR_Finger_Index1_link, origin xyz=0.0897 0.0101 0.023 rpy=0 -0.087266393 0, axis 0 0 1, limit lower=0 upper=1.5708 effort=-1 velocity=-1
- added joint HandR_Finger_Index2_joint: type revolute, parent HandR_Finger_Index1_link, child HandR_Finger_Index2_link, origin xyz=0.04524 0.0002 0 rpy=0 -0 0, axis 0 0 1, limit lower=0 upper=1.5708 effort=-1 velocity=-1
- added joint HandR_Finger_Middle1_joint: type revolute, parent ArmR_Wri2_link, child HandR_Finger_Middle1_link, origin xyz=0.0912501 0.01025 0.003 rpy=0 -0 0, axis 0 0 1, limit lower=0 upper=1.5708 effort=-1 velocity=-1
- added joint HandR_Finger_Middle2_joint: type revolute, parent HandR_Finger_Middle1_link, child HandR_Finger_Middle2_link, origin xyz=0.045 -0.003 0 rpy=0 -0 0, axis 0 0 1, limit lower=0 upper=1.5708 effort=-1 velocity=-1
- added joint HandR_Finger_Pinky1_joint: type revolute, parent ArmR_Wri2_link, child HandR_Finger_Pinky1_link, origin xyz=0.0888397 0.01024 -0.0311 rpy=0 0.174532697 0, axis 0 0 1, limit lower=0 upper=1.5708 effort=-1 velocity=-1
- added joint HandR_Finger_Pinky2_joint: type revolute, parent HandR_Finger_Pinky1_link, child HandR_Finger_Pinky2_link, origin xyz=0.027 0 0 rpy=0 -0 0, axis 0 0 1, limit lower=0 upper=1.5708 effort=-1 velocity=-1
- added joint HandR_Finger_Ring1_joint: type revolute, parent ArmR_Wri2_link, child HandR_Finger_Ring1_link, origin xyz=0.091442 0.01025 -0.0138 rpy=0 0.087266393 0, axis 0 0 1, limit lower=0 upper=1.5708 effort=-1 velocity=-1
- added joint HandR_Finger_Ring2_joint: type revolute, parent HandR_Finger_Ring1_link, child HandR_Finger_Ring2_link, origin xyz=0.04 0 0 rpy=0 -0 0, axis 0 0 1, limit lower=0 upper=1.5708 effort=-1 velocity=-1
- added joint HandR_Finger_Thumb1_joint: type revolute, parent ArmR_Wri2_link, child HandR_Finger_Thumb1_link, origin xyz=0.03527 0.01025 0.0091 rpy=1.57079637 -0 -1.57079637, axis 0 0 1, limit lower=0 upper=1.5708 effort=-1 velocity=-1
- added joint HandR_Finger_Thumb2_joint: type revolute, parent HandR_Finger_Thumb1_link, child HandR_Finger_Thumb2_link, origin xyz=0.00375 0.03 -0.00425 rpy=0 -1.57079625 0, axis 0 0 1, limit lower=0 upper=1.5708 effort=-1 velocity=-1
- added joint HandR_Finger_Thumb3_joint: type revolute, parent HandR_Finger_Thumb2_link, child HandR_Finger_Thumb3_link, origin xyz=0.0029 0.0293831 0 rpy=0 -0 0, axis 0 0 1, limit lower=0 upper=1.5708 effort=-1 velocity=-1
- added joint Head_1_joint: type revolute, parent Neck_3_link, child Head_1_link, origin xyz=0 0 0.1062 rpy=1.57079637 -0 -3.1415925, axis 0 0 1, limit lower=-0.174533 upper=0.610865 effort=-1 velocity=-1
- added joint Head_2_joint: type revolute, parent Head_1_link, child Head_2_link, origin xyz=0.00465 0 0 rpy=0 1.57079625 0, axis 0 0 1, limit lower=-0.349066 upper=0.349066 effort=-1 velocity=-1
- added joint LegL_Ank1_joint: type revolute, parent LegL_Knee_link, child LegL_Ank1_link, origin xyz=0 0 -0.4085 rpy=0 -1.57079625 0, axis 0 0 1, limit lower=-0.349066 upper=0.523599 effort=-1 velocity=-1
- added joint LegL_Ank2_joint: type revolute, parent LegL_Ank1_link, child LegL_Ank2_link, origin xyz=0 0 0 rpy=1.57079637 -0 0, axis 0 0 1, limit lower=-0.174533 upper=0.174533 effort=-1 velocity=-1
- added joint LegL_Heel_joint: type fixed, parent LegL_Ank2_link, child LegL_Heel_link, origin xyz=-0.0795 0 -0.053 rpy=-1.57079637 -0 0, axis 0 0 0, limit lower=0 upper=0 effort=-1 velocity=-1
- added joint LegL_Hip1_joint: type revolute, parent Root_link, child LegL_Hip1_link, origin xyz=0.124 0 -0.126 rpy=0 -0.615403175 0, axis 0 0 1, limit lower=-0.610865 upper=2.53073 effort=-1 velocity=-1
- added joint LegL_Hip2_joint: type revolute, parent LegL_Hip1_link, child LegL_Hip2_link, origin xyz=0 0 0 rpy=0.785398185 -1.57079625 0, axis 0 0 1, limit lower=0 upper=1.91986 effort=-1 velocity=-1
- added joint LegL_Hip3_joint: type revolute, parent LegL_Hip2_link, child LegL_Hip3_link, origin xyz=0 0 0 rpy=-1.57079637 -0 0, axis 0 0 1, limit lower=-0.523599 upper=1.91986 effort=-1 velocity=-1
- added joint LegL_Knee_joint: type revolute, parent LegL_Hip3_link, child LegL_Knee_link, origin xyz=-0.303136 -0.197542 0.173784 rpy=2.09439468 0.615402937 2.3561945, axis 1 0 0, limit lower=0 upper=1.74533 effort=-1 velocity=-1
- added joint LegL_Toe2_joint: type fixed, parent LegL_Ank2_link, child LegL_Toe2_link, origin xyz=-0.0742 -0.0006 0.1311 rpy=-1.13446438 -0 0, axis 0 0 0, limit lower=0 upper=0 effort=-1 velocity=-1
- added joint LegL_Toe_joint: type fixed, parent LegL_Ank2_link, child LegL_Toe_link, origin xyz=-0.07424 0.0244 0.13112 rpy=-1.57079637 -0 0, axis 0 0 0, limit lower=0 upper=0 effort=-1 velocity=-1
- added joint LegR_Ank1_joint: type revolute, parent LegR_Knee_link, child LegR_Ank1_link, origin xyz=0 0 0.4085 rpy=0 -1.57079625 0, axis 0 0 1, limit lower=-0.349066 upper=0.523599 effort=-1 velocity=-1
- added joint LegR_Ank2_joint: type revolute, parent LegR_Ank1_link, child LegR_Ank2_link, origin xyz=0 0 0 rpy=1.57079637 -0 0, axis 0 0 1, limit lower=-0.174533 upper=0.174533 effort=-1 velocity=-1
- added joint LegR_Heel_joint: type fixed, parent LegR_Ank2_link, child LegR_Heel_link, origin xyz=0.07945 0 0.0529 rpy=0 -0 0, axis 0 0 0, limit lower=0 upper=0 effort=-1 velocity=-1
- added joint LegR_Hip1_joint: type revolute, parent Root_link, child LegR_Hip1_link, origin xyz=-0.124 0 -0.126 rpy=-3.1415925 0.615403175 0, axis 0 0 1, limit lower=-0.610865 upper=2.53073 effort=-1 velocity=-1
- added joint LegR_Hip2_joint: type revolute, parent LegR_Hip1_link, child LegR_Hip2_link, origin xyz=0 0 0 rpy=0.785398185 -1.57079625 0, axis 0 0 1, limit lower=0 upper=1.91986 effort=-1 velocity=-1
- added joint LegR_Hip3_joint: type revolute, parent LegR_Hip2_link, child LegR_Hip3_link, origin xyz=0 0 0 rpy=-1.57079637 -0 0, axis 0 0 1, limit lower=-0.523599 upper=1.91986 effort=-1 velocity=-1
- added joint LegR_Knee_joint: type revolute, parent LegR_Hip3_link, child LegR_Knee_link, origin xyz=0.3031 0.1975 -0.1738 rpy=2.09439468 0.615402937 2.3561945, axis 1 0 0, limit lower=0 upper=1.74533 effort=-1 velocity=-1
- added joint LegR_Toe2_joint: type fixed, parent LegR_Ank2_link, child LegR_Toe2_link, origin xyz=0.0743 0.0006 -0.1312 rpy=-1.13446438 -0 0, axis 0 0 0, limit lower=0 upper=0 effort=-1 velocity=-1
- added joint LegR_Toe_joint: type fixed, parent LegR_Ank2_link, child LegR_Toe_link, origin xyz=0.0743 -0.0254 -0.13117 rpy=3.14159274 -1.50996001e-07 3.14159274, axis 0 0 0, limit lower=0 upper=0 effort=-1 velocity=-1
- added joint Neck_1_joint: type revolute, parent Torso_Pitch_link, child Neck_1_link, origin xyz=0 0.3073 0 rpy=0 -0 -1.57079637, axis 0 0 1, limit lower=-0.785398 upper=0.610865 effort=-1 velocity=-1
- added joint Neck_2_joint: type revolute, parent Neck_1_link, child Neck_2_link, origin xyz=0 0 0 rpy=-1.57079637 1.57079625 0, axis 0 0 1, limit lower=-1.22173 upper=1.22173 effort=-1 velocity=-1
- added joint Neck_3_joint: type revolute, parent Neck_2_link, child Neck_3_link, origin xyz=0 0.0338 0 rpy=-1.57079637 1.57079625 0, axis 0 0 1, limit lower=-1.5708 upper=1.5708 effort=-1 velocity=-1
- added joint Root_joint: type fixed, parent root, child Root_link, origin xyz=0 0 0 rpy=0 -0 0, axis 0 0 0, limit lower=0 upper=0 effort=-1 velocity=-1
- added joint Torso_Pitch_joint: type revolute, parent Torso_Yaw_link, child Torso_Pitch_link, origin xyz=0 0 0.099879 rpy=1.57079637 -0 1.57079637, axis 0 0 1, limit lower=-0.785398 upper=0.785398 effort=-1 velocity=-1
- added joint Torso_Yaw_joint: type revolute, parent Root_link, child Torso_Yaw_link, origin xyz=0 0 0 rpy=0 -0 0, axis 0 0 1, limit lower=-1.5708 upper=1.5708 effort=-1 velocity=-1
- joint HandL_TCP_joint: parent ArmL_Wri2_joint_link -> ArmL_Wri2_link
- joint HandR_TCP_joint: parent ArmR_Wri2_joint_link -> ArmR_Wri2_link
- joint LegL_Ank2_body_joint: parent LegL_Ank2_joint_link -> LegL_Ank2_link
- joint LegL_TCP_joint: parent LegL_Ank2_joint_link -> LegL_Ank2_link
- joint LegR_Ank2_body_joint: parent LegR_Ank2_joint_link -> LegR_Ank2_link
- joint LegR_TCP_joint: parent LegR_Ank2_joint_link -> LegR_Ank2_link
- joint Pelvis_joint: parent Root_joint_link -> Root_link
- joint TorsoCenter_joint: parent Torso_Pitch_joint_link -> Torso_Pitch_link
