Commit message: Update Armar4 model for use in qt3d

File: data/robots/Armar4/urdf/Armar4.urdf (robot description, URDF)
Before this commit: robot Armar4, 80 links, 79 joints
Links:
- link ArmL_Elb1_link: geometry collision mesh filename=stl/ArmL_Elb1_joint_col.stl scale=1 1 1; visual mesh filename=stl/ArmL_Elb1_joint_visu.dae scale=1 1 1
- link ArmL_Elb2_link: geometry collision mesh filename=stl/ArmL_Elb2_joint_col.stl scale=1 1 1; visual mesh filename=stl/ArmL_Elb2_joint_visu.dae scale=1 1 1
- link ArmL_Sho1_link: geometry collision mesh filename=stl/ArmL_Sho1_joint_col.stl scale=1 1 1; visual mesh filename=stl/ArmL_Sho1_joint_visu.dae scale=1 1 1
- link ArmL_Sho2_link: geometry collision mesh filename=stl/ArmL_Sho2_joint_col.stl scale=1 1 1; visual mesh filename=stl/ArmL_Sho2_joint_visu.dae scale=1 1 1
- link ArmL_Sho3_link: geometry collision mesh filename=stl/ArmL_Sho3_joint_col.stl scale=1 1 1; visual mesh filename=stl/ArmL_Sho3_joint_visu.dae scale=1 1 1
- link ArmL_Sho4_link: geometry collision mesh filename=stl/ArmL_Sho4_joint_col.stl scale=1 1 1; visual mesh filename=stl/ArmL_Sho4_joint_visu.dae scale=1 1 1
- link ArmL_Wri1_link: geometry collision mesh filename=stl/sphere10.stl scale=1 1 1; visual mesh filename=stl/ArmL_Wri1_joint_visu.dae scale=1 1 1
- link ArmL_Wri2_link: geometry collision mesh filename=stl/ArmL_Wri2_joint_col.stl scale=1 1 1; visual mesh filename=stl/ArmL_Wri2_joint_visu.dae scale=1 1 1
- link Torso_Pitch_link: geometry collision mesh filename=stl/Torso_Pitch_joint_col.stl scale=1 1 1; visual mesh filename=stl/Torso2_joint_visu.dae scale=1 1 1

Commit message: Updates to URDF model of Armar4

File: data/robots/Armar4/urdf/Armar4.urdf (robot description, URDF)
Before this commit: robot Armar4, 80 links, 79 joints
Links:
- link ArmL_Elb1_link: geometry collision mesh filename=stl/ArmL_Elb1_joint_col.stl scale=1000 1000 1000; visual mesh filename=stl/ArmL_Elb1_joint_visu.dae scale=1000 1000 1000
- link ArmL_Elb2_link: geometry collision mesh filename=stl/ArmL_Elb2_joint_col.stl scale=1000 1000 1000; visual mesh filename=stl/ArmL_Elb2_joint_visu.dae scale=1000 1000 1000
- link ArmL_Sho1_link: geometry collision mesh filename=stl/ArmL_Sho1_joint_col.stl scale=1000 1000 1000; visual mesh filename=stl/ArmL_Sho1_joint_visu.dae scale=1000 1000 1000
- link ArmL_Sho2_link: geometry collision mesh filename=stl/ArmL_Sho2_joint_col.stl scale=1000 1000 1000; visual mesh filename=stl/ArmL_Sho2_joint_visu.dae scale=1000 1000 1000
- link ArmL_Sho3_link: geometry collision mesh filename=stl/ArmL_Sho3_joint_col.stl scale=1000 1000 1000; visual mesh filename=stl/ArmL_Sho3_joint_visu.dae scale=1000 1000 1000
- link ArmL_Sho4_link: geometry collision mesh filename=stl/ArmL_Sho4_joint_col.stl scale=1000 1000 1000; visual mesh filename=stl/ArmL_Sho4_joint_visu.dae scale=1000 1000 1000
- link ArmL_Wri1_link: geometry collision mesh filename=stl/sphere10.stl scale=1000 1000 1000; visual mesh filename=stl/ArmL_Wri1_joint_visu.dae scale=1000 1000 1000
- link ArmL_Wri2_link: geometry collision mesh filename=stl/ArmL_Wri2_joint_col.stl scale=1000 1000 1000; visual mesh filename=stl/ArmL_Wri2_joint_visu.dae scale=1000 1000 1000
- link ArmR_Elb1_link: geometry collision mesh filename=stl/ArmR_Elb1_joint_col.stl scale=1000 1000 1000; visual mesh filename=stl/ArmR_Elb1_joint_visu.dae scale=1000 1000 1000
- link ArmR_Elb2_link: geometry collision mesh filename=stl/ArmR_Elb2_joint_col.stl scale=1000 1000 1000; visual mesh filename=stl/ArmR_Elb2_joint_visu.dae scale=1000 1000 1000
- link ArmR_Sho1_link: geometry collision mesh filename=stl/ArmR_Sho1_joint_col.stl scale=1000 1000 1000; visual mesh filename=stl/ArmR_Sho1_joint_visu.dae scale=1000 1000 1000
- link ArmR_Sho2_link: geometry collision mesh filename=stl/ArmR_Sho2_joint_col.stl scale=1000 1000 1000; visual mesh filename=stl/ArmR_Sho2_joint_visu.dae scale=1000 1000 1000
- link ArmR_Sho3_link: geometry collision mesh filename=stl/ArmR_Sho3_joint_col.stl scale=1000 1000 1000; visual mesh filename=stl/ArmR_Sho3_joint_visu.dae scale=1000 1000 1000
- link ArmR_Sho4_link: geometry collision mesh filename=stl/ArmR_Sho4_joint_col.stl scale=1000 1000 1000; visual mesh filename=stl/ArmR_Sho4_joint_visu.dae scale=1000 1000 1000
- link ArmR_Wri1_link: geometry collision mesh filename=stl/sphere10.stl scale=1000 1000 1000; visual mesh filename=stl/ArmR_Wri1_joint_visu.dae scale=1000 1000 1000
- link ArmR_Wri2_link: geometry collision mesh filename=stl/ArmR_Wri2_joint_col.stl scale=1000 1000 1000; visual mesh filename=stl/ArmR_Wri2_joint_visu.dae scale=1000 1000 1000
- link EyeL_1_link: geometry collision mesh filename=stl/EyeL_1_joint_visu.stl scale=1000 1000 1000; visual mesh filename=stl/EyeL_1_joint_visu.dae scale=1000 1000 1000
- link EyeL_2_link: geometry collision mesh filename=stl/EyeL_2_joint_col.stl scale=1000 1000 1000; visual mesh filename=stl/EyeL_2_joint_visu.dae scale=1000 1000 1000
- link EyeR_1_link: geometry collision mesh filename=stl/EyeR_1_joint_visu.stl scale=1000 1000 1000; visual mesh filename=stl/EyeR_1_joint_visu.dae scale=1000 1000 1000
- link EyeR_2_link: geometry collision mesh filename=stl/EyeR_2_joint_visu.stl scale=1000 1000 1000; visual mesh filename=stl/EyeR_2_joint_visu.dae scale=1000 1000 1000
- link HandL_Finger_Index1_link: geometry collision mesh filename=stl/HandL_Finger_Index1_joint_col.stl scale=1000 1000 1000; visual mesh filename=stl/HandL_Finger_Index1_joint_visu.stl scale=1000 1000 1000
- link HandL_Finger_Index2_link: geometry collision mesh filename=stl/HandL_Finger_Index2_joint_col.stl scale=1000 1000 1000; visual mesh filename=stl/HandL_Finger_Index2_joint_visu.stl scale=1000 1000 1000
- link HandL_Finger_Middle1_link: geometry collision mesh filename=stl/HandL_Finger_Middle1_joint_col.stl scale=1000 1000 1000; visual mesh filename=stl/HandL_Finger_Middle1_joint_visu.stl scale=1000 1000 1000
- link HandL_Finger_Middle2_link: geometry collision mesh filename=stl/HandL_Finger_Middle2_joint_col.stl scale=1000 1000 1000; visual mesh filename=stl/HandL_Finger_Middle2_joint_visu.stl scale=1000 1000 1000
- link HandL_Finger_Pinky1_link: geometry collision mesh filename=stl/HandL_Finger_Pinky1_joint_col.stl scale=1000 1000 1000; visual mesh filename=stl/HandL_Finger_Pinky1_joint_visu.stl scale=1000 1000 1000
- link HandL_Finger_Pinky2_link: geometry collision mesh filename=stl/HandL_Finger_Pinky2_joint_col.stl scale=1000 1000 1000; visual mesh filename=stl/HandL_Finger_Pinky2_joint_visu.stl scale=1000 1000 1000
- link HandL_Finger_Ring1_link: geometry collision mesh filename=stl/HandL_Finger_Ring1_joint_col.stl scale=1000 1000 1000; visual mesh filename=stl/HandL_Finger_Ring1_joint_visu.stl scale=1000 1000 1000
- link HandL_Finger_Ring2_link: geometry collision mesh filename=stl/HandL_Finger_Ring2_joint_col.stl scale=1000 1000 1000; visual mesh filename=stl/HandL_Finger_Ring2_joint_visu.stl scale=1000 1000 1000
- link HandL_Finger_Thumb1_link: geometry collision mesh filename=stl/HandL_Finger_Thumb1_joint_col.stl scale=1000 1000 1000; visual mesh filename=stl/HandL_Finger_Thumb1_joint_visu.stl scale=1000 1000 1000
- link HandL_Finger_Thumb2_link: geometry collision mesh filename=stl/HandL_Finger_Thumb2_joint_col.stl scale=1000 1000 1000; visual mesh filename=stl/HandL_Finger_Thumb2_joint_visu.stl scale=1000 1000 1000
- link HandL_Finger_Thumb3_link: geometry collision mesh filename=stl/HandL_Finger_Thumb3_joint_col.stl scale=1000 1000 1000; visual mesh filename=stl/HandL_Finger_Thumb3_joint_visu.stl scale=1000 1000 1000
- link HandR_Finger_Index1_link: geometry collision mesh filename=stl/HandR_Finger_Index1_joint_col.stl scale=1000 1000 1000; visual mesh filename=stl/HandR_Finger_Index1_joint_visu.stl scale=1000 1000 1000
- link HandR_Finger_Index2_link: geometry collision mesh filename=stl/HandR_Finger_Index2_joint_col.stl scale=1000 1000 1000; visual mesh filename=stl/HandR_Finger_Index2_joint_visu.stl scale=1000 1000 1000
- link HandR_Finger_Middle1_link: geometry collision mesh filename=stl/HandR_Finger_Middle1_joint_col.stl scale=1000 1000 1000; visual mesh filename=stl/HandR_Finger_Middle1_joint_visu.stl scale=1000 1000 1000
- link HandR_Finger_Middle2_link: geometry collision mesh filename=stl/HandR_Finger_Middle2_joint_col.stl scale=1000 1000 1000; visual mesh filename=stl/HandR_Finger_Middle2_joint_visu.stl scale=1000 1000 1000
- link HandR_Finger_Pinky1_link: geometry collision mesh filename=stl/HandR_Finger_Pinky1_joint_col.stl scale=1000 1000 1000; visual mesh filename=stl/HandR_Finger_Pinky1_joint_visu.stl scale=1000 1000 1000
- link HandR_Finger_Pinky2_link: geometry collision mesh filename=stl/HandR_Finger_Pinky2_joint_col.stl scale=1000 1000 1000; visual mesh filename=stl/HandR_Finger_Pinky2_joint_visu.stl scale=1000 1000 1000
- link HandR_Finger_Ring1_link: geometry collision mesh filename=stl/HandR_Finger_Ring1_joint_col.stl scale=1000 1000 1000; visual mesh filename=stl/HandR_Finger_Ring1_joint_visu.stl scale=1000 1000 1000
- link HandR_Finger_Ring2_link: geometry collision mesh filename=stl/HandR_Finger_Ring2_joint_col.stl scale=1000 1000 1000; visual mesh filename=stl/HandR_Finger_Ring2_joint_visu.stl scale=1000 1000 1000
- link HandR_Finger_Thumb1_link: geometry collision mesh filename=stl/HandR_Finger_Thumb1_joint_col.stl scale=1000 1000 1000; visual mesh filename=stl/HandR_Finger_Thumb1_joint_visu.stl scale=1000 1000 1000
- link HandR_Finger_Thumb2_link: geometry collision mesh filename=stl/HandR_Finger_Thumb2_joint_col.stl scale=1000 1000 1000; visual mesh filename=stl/HandR_Finger_Thumb2_joint_visu.stl scale=1000 1000 1000
- link HandR_Finger_Thumb3_link: geometry collision mesh filename=stl/HandR_Finger_Thumb3_joint_col.stl scale=1000 1000 1000; visual mesh filename=stl/HandR_Finger_Thumb3_joint_visu.stl scale=1000 1000 1000
- link Head_1_link: geometry collision mesh filename=stl/Head_1_joint_col.stl scale=1000 1000 1000; visual mesh filename=stl/Head_1_joint_visu.dae scale=1000 1000 1000
- link Head_2_link: geometry collision mesh filename=stl/Head_2_joint_col.stl scale=1000 1000 1000; visual mesh filename=stl/Head_2_joint_visu.dae scale=1000 1000 1000
- link LegL_Ank1_link: geometry collision mesh filename=stl/sphere10.stl scale=1000 1000 1000
- link LegL_Ank2_body_link: geometry collision mesh filename=stl/LegL_Ank2_joint_col.stl scale=1000 1000 1000; visual mesh filename=stl/LegL_Ank2_joint_visu.stl scale=1000 1000 1000
- link LegL_Heel_link: geometry collision mesh filename=stl/LegL_Heel_joint_visu.stl scale=1000 1000 1000; visual mesh filename=stl/LegL_Heel_joint_visu.stl scale=1000 1000 1000
- link LegL_Hip1_link: geometry collision mesh filename=stl/LegL_Hip1_joint_col.stl scale=1000 1000 1000; visual mesh filename=stl/LegL_Hip1_joint_visu.stl scale=1000 1000 1000
- link LegL_Hip2_link: geometry collision mesh filename=stl/LegL_Hip2_joint_col.stl scale=1000 1000 1000; visual mesh filename=stl/LegL_Hip2_joint_visu.stl scale=1000 1000 1000
- link LegL_Hip3_link: geometry collision mesh filename=stl/LegL_Hip3_joint_col.stl scale=1000 1000 1000; visual mesh filename=stl/LegL_Hip3_joint_visu.stl scale=1000 1000 1000
- link LegL_Knee_link: geometry collision mesh filename=stl/LegL_Knee_joint_col.stl scale=1000 1000 1000; visual mesh filename=stl/LegL_Knee_joint_visu.stl scale=1000 1000 1000
- link LegL_Toe2_link: geometry collision mesh filename=stl/LegL_Toe2_joint_visu.stl scale=1000 1000 1000; visual mesh filename=stl/LegL_Toe2_joint_visu.stl scale=1000 1000 1000
- link LegL_Toe_link: geometry collision mesh filename=stl/LegL_Toe_joint_visu.stl scale=1000 1000 1000; visual mesh filename=stl/LegL_Toe_joint_visu.stl scale=1000 1000 1000
- link LegR_Ank1_link: geometry collision mesh filename=stl/sphere10.stl scale=1000 1000 1000
- link LegR_Ank2_body_link: geometry collision mesh filename=stl/LegR_Ank2_joint_col.stl scale=1000 1000 1000; visual mesh filename=stl/LegR_Ank2_joint_visu.stl scale=1000 1000 1000
- link LegR_Heel_link: geometry collision mesh filename=stl/LegR_Heel_joint_visu.stl scale=1000 1000 1000; visual mesh filename=stl/LegR_Heel_joint_visu.stl scale=1000 1000 1000
- link LegR_Hip1_link: geometry collision mesh filename=stl/LegR_Hip1_joint_col.stl scale=1000 1000 1000; visual mesh filename=stl/LegR_Hip1_joint_visu.stl scale=1000 1000 1000
- link LegR_Hip2_link: geometry collision mesh filename=stl/LegR_Hip2_joint_col.stl scale=1000 1000 1000; visual mesh filename=stl/LegR_Hip2_joint_visu.stl scale=1000 1000 1000
- link LegR_Hip3_link: geometry collision mesh filename=stl/LegR_Hip3_joint_col.stl scale=1000 1000 1000; visual mesh filename=stl/LegR_Hip3_joint_visu.stl scale=1000 1000 1000
- link LegR_Knee_link: geometry collision mesh filename=stl/LegR_Knee_joint_col.stl scale=1000 1000 1000; visual mesh filename=stl/LegR_Knee_joint_visu.stl scale=1000 1000 1000
- link LegR_Toe2_link: geometry collision mesh filename=stl/LegR_Toe2_joint_visu.stl scale=1000 1000 1000; visual mesh filename=stl/LegR_Toe2_joint_visu.stl scale=1000 1000 1000
- link LegR_Toe_link: geometry collision mesh filename=stl/LegR_Toe_joint_visu.stl scale=1000 1000 1000; visual mesh filename=stl/LegR_Toe_joint_visu.stl scale=1000 1000 1000
- link Neck_1_link: geometry collision mesh filename=stl/Neck_1_joint_col.stl scale=1000 1000 1000; visual mesh filename=stl/Neck_1_joint_visu.dae scale=1000 1000 1000
- link Neck_2_link: geometry collision mesh filename=stl/Neck_2_joint_col.stl scale=1000 1000 1000; visual mesh filename=stl/Neck_2_joint_visu.dae scale=1000 1000 1000
- link Neck_3_link: geometry collision mesh filename=stl/Neck_3_joint_col.stl scale=1000 1000 1000; visual mesh filename=stl/Neck_3_joint_visu.dae scale=1000 1000 1000
- link Root_link: geometry collision mesh filename=stl/Root_joint_col.stl scale=1000 1000 1000; visual mesh filename=stl/Root_joint_visu.stl scale=1000 1000 1000
- link Torso_Pitch_link: geometry collision mesh filename=stl/Torso_Pitch_joint_col.stl scale=1000 1000 1000; visual mesh filename=stl/Torso2_joint_visu.dae scale=1000 1000 1000
- link Torso_Yaw_link: geometry collision mesh filename=stl/Torso_Yaw_joint_col.stl scale=1000 1000 1000; visual mesh filename=stl/Torso_Yaw_joint_visu.stl scale=1000 1000 1000
