Commit message: added armar3 iv-meshes (fullmodel)

File: data/robots/Armar3/urdf/Armar3.urdf (robot description, URDF)
Before this commit: robot Armar3, 108 links, 107 joints
Links:
- link Elbow L_link: geometry collision mesh filename=stl/elbow_l.stl scale=1 1 1; visual mesh filename=fullmodel/elbow_l.iv scale=1 1 1
- link Elbow R_link: geometry collision mesh filename=stl/elbow_r.stl scale=1 1 1; visual mesh filename=fullmodel/elbow_r.iv scale=1 1 1
- link Eye_Left_link: geometry collision mesh filename=stl/cyl1.stl scale=1 1 1; visual mesh filename=fullmodel/eye_l.iv scale=1 1 1
- link Eye_Right_link: geometry collision mesh filename=stl/cyl1.stl scale=1 1 1; visual mesh filename=fullmodel/eye_r.iv scale=1 1 1
- link Hand Palm 1 L_link: geometry collision mesh filename=stl/palm1_l.stl scale=1 1 1; visual mesh filename=fullmodel/palm1_l.iv scale=1 1 1
- link Hand Palm 1 R_link: geometry collision mesh filename=stl/palm1_r.stl scale=1 1 1; visual mesh filename=fullmodel/palm1_r.iv scale=1 1 1
- link Hand Palm 2 L_link: geometry collision mesh filename=stl/palm2_l.stl scale=1 1 1; visual mesh filename=fullmodel/palm2_l.iv scale=1 1 1
- link Hand Palm 2 R_link: geometry collision mesh filename=stl/palm2_r.stl scale=1 1 1; visual mesh filename=fullmodel/palm2_r.iv scale=1 1 1
- link Head Base_link: geometry collision mesh filename=stl/head_base.stl scale=1 1 1; visual mesh filename=fullmodel/head_base.iv scale=1 1 1
- link Head_Tilt_link: geometry collision mesh filename=stl/head.stl scale=1 1 1; visual mesh filename=fullmodel/head.iv scale=1 1 1
- link Hip Pitch_link: geometry collision mesh filename=stl/platform_pitch_link.stl scale=1 1 1; visual mesh filename=fullmodel/platform_pitch_link.iv scale=1 1 1
- link Hip Roll_link: geometry collision mesh filename=stl/platform_roll_link.stl scale=1 1 1; visual mesh filename=fullmodel/platform_roll_link.iv scale=1 1 1
- link Hip Yaw_link: geometry collision mesh filename=stl/torso.stl scale=1 1 1; visual mesh filename=fullmodel/torso.iv scale=1 1 1
- link Index L J0_link: geometry collision mesh filename=stl/index_l1.stl scale=1 1 1; visual mesh filename=fullmodel/index_l1.iv scale=1 1 1
- link Index L J1_link: geometry collision mesh filename=stl/index_l2.stl scale=1 1 1; visual mesh filename=fullmodel/index_l2.iv scale=1 1 1
- link Index R J0_link: geometry collision mesh filename=stl/index_r1.stl scale=1 1 1; visual mesh filename=fullmodel/index_r1.iv scale=1 1 1
- link Index R J1_link: geometry collision mesh filename=stl/index_r2.stl scale=1 1 1; visual mesh filename=fullmodel/index_r2.iv scale=1 1 1
- link Jaw_link: geometry visual mesh filename=fullmodel/jaw.iv scale=1 1 1
- link Lid Left Bottom_link: geometry visual mesh filename=fullmodel/lid_l_bottom.iv scale=1 1 1
- link Lid Left Top_link: geometry visual mesh filename=fullmodel/lid_l_top.iv scale=1 1 1
- link Lid Right Bottom_link: geometry visual mesh filename=fullmodel/lid_r_bottom.iv scale=1 1 1
- link Lid Right Top_link: geometry visual mesh filename=fullmodel/lid_r_top.iv scale=1 1 1
- link Middle L J0_link: geometry collision mesh filename=stl/middle_l1.stl scale=1 1 1; visual mesh filename=fullmodel/middle_l1.iv scale=1 1 1
- link Middle L J1_link: geometry collision mesh filename=stl/middle_l2.stl scale=1 1 1; visual mesh filename=fullmodel/middle_l2.iv scale=1 1 1
- link Middle R J0_link: geometry collision mesh filename=stl/middle_r1.stl scale=1 1 1; visual mesh filename=fullmodel/middle_r1.iv scale=1 1 1
- link Middle R J1_link: geometry collision mesh filename=stl/middle_r2.stl scale=1 1 1; visual mesh filename=fullmodel/middle_r2.iv scale=1 1 1
- link Neck_1_Pitch_link: geometry collision mesh filename=stl/neck_pitch_link.stl scale=1 1 1; visual mesh filename=fullmodel/neck_pitch_link.iv scale=1 1 1
- link Neck_2_Roll_link: geometry collision mesh filename=stl/neck_roll_link.stl scale=1 1 1; visual mesh filename=fullmodel/neck_roll_link.iv scale=1 1 1
- link Neck_3_Yaw_link: geometry collision mesh filename=stl/neck_yaw_link.stl scale=1 1 1; visual mesh filename=fullmodel/neck_yaw_link.iv scale=1 1 1
- link Pinky L J0_link: geometry collision mesh filename=stl/pinky_l1.stl scale=1 1 1; visual mesh filename=fullmodel/pinky_l1.iv scale=1 1 1
- link Pinky L J1_link: geometry collision mesh filename=stl/pinky_l2.stl scale=1 1 1; visual mesh filename=fullmodel/pinky_l2.iv scale=1 1 1
- link Pinky R J0_link: geometry collision mesh filename=stl/pinky_r1.stl scale=1 1 1; visual mesh filename=fullmodel/pinky_r1.iv scale=1 1 1
- link Pinky R J1_link: geometry collision mesh filename=stl/pinky_r2.stl scale=1 1 1; visual mesh filename=fullmodel/pinky_r2.iv scale=1 1 1
- link Platform_link: geometry collision mesh filename=stl/platform.stl scale=1 1 1; visual mesh filename=fullmodel/platform.iv scale=1 1 1
- link Ring L J0_link: geometry collision mesh filename=stl/ring_l1.stl scale=1 1 1; visual mesh filename=fullmodel/ring_l1.iv scale=1 1 1
- link Ring L J1_link: geometry collision mesh filename=stl/ring_l2.stl scale=1 1 1; visual mesh filename=fullmodel/ring_l2.iv scale=1 1 1
- link Ring R J0_link: geometry collision mesh filename=stl/ring_r1.stl scale=1 1 1; visual mesh filename=fullmodel/ring_r1.iv scale=1 1 1
- link Ring R J1_link: geometry collision mesh filename=stl/ring_r2.stl scale=1 1 1; visual mesh filename=fullmodel/ring_r2.iv scale=1 1 1
- link Shoulder 1 L_link: geometry collision mesh filename=stl/shoulder_l.stl scale=1 1 1; visual mesh filename=fullmodel/shoulder_l.iv scale=1 1 1
- link Shoulder 1 R_link: geometry collision mesh filename=stl/shoulder_r.stl scale=1 1 1; visual mesh filename=fullmodel/shoulder_r.iv scale=1 1 1
- link Shoulder 2 L_link: geometry collision mesh filename=stl/shoulder2_l_rot.stl scale=1 1 1; visual mesh filename=fullmodel/shoulder2_l_rot.iv scale=1 1 1
- link Shoulder 2 R_link: geometry collision mesh filename=stl/shoulder2_r_rot.stl scale=1 1 1; visual mesh filename=fullmodel/shoulder2_r_rot.iv scale=1 1 1
- link Thumb L J0_link: geometry collision mesh filename=stl/thumb_l1.stl scale=1 1 1; visual mesh filename=fullmodel/thumb_l1.iv scale=1 1 1
- link Thumb L J1_link: geometry collision mesh filename=stl/thumb_l2.stl scale=1 1 1; visual mesh filename=fullmodel/thumb_l2.iv scale=1 1 1
- link Thumb R J0_link: geometry collision mesh filename=stl/thumb_r1.stl scale=1 1 1; visual mesh filename=fullmodel/thumb_r1.iv scale=1 1 1
- link Thumb R J1_link: geometry collision mesh filename=stl/thumb_r2.stl scale=1 1 1; visual mesh filename=fullmodel/thumb_r2.iv scale=1 1 1
- link Underarm L_link: geometry collision mesh filename=stl/underarm_l.stl scale=1 1 1; visual mesh filename=fullmodel/underarm_l.iv scale=1 1 1
- link Underarm R_link: geometry collision mesh filename=stl/underarm_r.stl scale=1 1 1; visual mesh filename=fullmodel/underarm_r.iv scale=1 1 1
- link Upperarm L_link: geometry collision mesh filename=stl/upperarm_l.stl scale=1 1 1; visual mesh filename=fullmodel/upperarm_l.iv scale=1 1 1

Commit message: CoinVisualizationFactory now renders attachements, too.

File: data/robots/Armar3/urdf/Armar3.urdf (robot description, URDF)
Before this commit: robot Armar3, 108 links, 107 joints
Links:
- link Upperarm R_link: geometry collision mesh filename=stl/upperarm_r.stl scale=1 1 1; visual mesh filename=fullmodel/upperarm_r.iv scale=1 1 1

Commit message: fix Armar-3 platform joints scene updates

File: data/robots/Armar3/urdf/Armar3.urdf (robot description, URDF)
Before this commit: robot Armar3, 108 links, 107 joints
Joints:
- joint X_Platform_joint: axis 0 0 0 -> 0 0 -1; limit lower=0 upper=0 effort=-1 velocity=-1 -> lower=-0 upper=5000 effort=-1 velocity=-1; type fixed -> prismatic
- joint Y_Platform_joint: axis 0 0 0 -> 1 0 0; limit lower=0 upper=0 effort=-1 velocity=-1 -> lower=0 upper=10000 effort=-1 velocity=-1; type fixed -> prismatic
