Commit message: remove '_joint' from Armar3 joints in model description fix frame loading

File: data/robots/Armar3/urdf/Armar3.urdf (robot description, URDF)
Before this commit: robot Armar3, 108 links, 107 joints
Joints:
- removed joint Armar3_Base_joint
- removed joint Cameras_joint
- removed joint Center of Arms_joint
- removed joint DepthCameraSim_joint
- removed joint DepthCamera_joint
- removed joint Dummy_Platform_joint
- removed joint Elbow L_joint
- removed joint Elbow R_joint
- removed joint EndArmL_joint
- removed joint EndArmR_joint
- removed joint EyeLeftCameraPreTransformation_joint
- removed joint EyeLeftCameraSim_joint
- removed joint EyeLeftCamera_joint
- removed joint EyeRightCameraPreTransformation_joint
- removed joint EyeRightCameraSim_joint
- removed joint EyeRightCamera_joint
- removed joint Eye_Left_Dummy_joint
- removed joint Eye_Left_joint
- removed joint Eye_Right_Dummy_joint
- removed joint Eye_Right_joint
- removed joint GCP L_joint
- removed joint GCP R_joint
- removed joint Hand L Base_joint
- removed joint Hand Palm 1 L_joint
- removed joint Hand Palm 1 R_joint
- removed joint Hand Palm 2 L_joint
- removed joint Hand Palm 2 R_joint
- removed joint Hand R Base_joint
- removed joint Head Base_joint
- removed joint Head Center1_joint
- removed joint Head Center_joint
- removed joint HeadIMU_joint
- removed joint HeadMotionMeasurementTCP_joint
- removed joint Head_Tilt_joint
- removed joint Hip Pitch_joint
- removed joint Hip Roll_joint
- removed joint Hip Yaw_joint
- removed joint Index L J0_joint
- removed joint Index L J1_joint
- removed joint Index L_joint
- removed joint Index R Fingertip_joint
- removed joint Index R J0_joint
- removed joint Index R J1_joint
- removed joint Index R_joint
- removed joint Jaw_joint
- removed joint Kinect_joint
- removed joint Left Arm Base_joint
- removed joint Lid Left Bottom_joint
- removed joint Lid Left Top_joint
- removed joint Lid Right Bottom_joint
- removed joint Lid Right Top_joint
- removed joint Marker L_joint
- removed joint Marker R_joint
- removed joint Middle L J0_joint
- removed joint Middle L J1_joint
- removed joint Middle L_joint
- removed joint Middle R Fingertip_joint
- removed joint Middle R J0_joint
- removed joint Middle R J1_joint
- removed joint Middle R_joint
- removed joint Neck_1_Pitch_joint
- removed joint Neck_2_Roll_joint
- removed joint Neck_3_Yaw_joint
- removed joint Pinky L J0_joint
- removed joint Pinky L J1_joint
- removed joint Pinky L_joint
- removed joint Pinky R J0_joint
- removed joint Pinky R J1_joint
- removed joint Pinky R_joint
- removed joint Platform_joint
- removed joint Right Arm Base_joint
- removed joint Ring L J0_joint
- removed joint Ring L J1_joint
- removed joint Ring L_joint
- removed joint Ring R J0_joint
- removed joint Ring R J1_joint
- removed joint Ring R_joint
- removed joint Shoulder 1 L_joint
- removed joint Shoulder 1 R_joint
- removed joint Shoulder 2 L_joint
- removed joint Shoulder 2 R_joint
- removed joint TCP L_joint
- removed joint TCP R_joint
- removed joint Thumb L J0_joint
- removed joint Thumb L J1_joint
- removed joint Thumb L_joint
- removed joint Thumb R Fingertip_joint
- removed joint Thumb R J0_joint
- removed joint Thumb R J1_joint
- removed joint Thumb R_joint
- removed joint TrafoToHead_joint
- removed joint TrafoToLeftArm_joint
- removed joint TrafoToRightArm_joint
- removed joint Underarm L_joint
- removed joint Underarm R_joint
- removed joint Upperarm L_joint
- removed joint Upperarm R_joint
- removed joint VirtualCentralGaze_joint
- removed joint Wrist 1 L_joint
- removed joint Wrist 1 R_joint
- removed joint Wrist 2 L_joint
- removed joint Wrist 2 R_joint
- removed joint X_Platform_joint
- removed joint Y_Platform_joint
- removed joint Yaw_Platform_joint
- removed joint left_hand_configuration_actual_float_joint
- removed joint right_hand_configuration_actual_float_joint
- added joint Armar3_Base: type fixed, parent root, child Armar3_Base_link, origin xyz=0 0 0 rpy=0 -0 0, axis 0 0 0, limit lower=0 upper=0 effort=-1 velocity=-1
- added joint Cameras: type revolute, parent Head Center_link, child Cameras_link, origin xyz=0.1 0 0 rpy=0 -0 0, axis 0 0 -1, limit lower=-0.349066 upper=0.0872665 effort=-1 velocity=1
- added joint Center of Arms: type fixed, parent Hip Yaw_link, child Center of Arms_link, origin xyz=0 -0.035 0.485 rpy=0 -0 0, axis 0 0 0, limit lower=0 upper=0 effort=-1 velocity=-1
- added joint DepthCamera: type fixed, parent Head Center_link, child DepthCamera_link, origin xyz=0.105 0.07 0 rpy=1.66814637 1.57079613 1.94739902, axis 0 0 0, limit lower=0 upper=0 effort=-1 velocity=-1
- added joint DepthCameraSim: type fixed, parent Head Center_link, child DepthCameraSim_link, origin xyz=0.105 0.07 0 rpy=1.57079637 -1.09154875e-07 1.93207955, axis 0 0 0, limit lower=0 upper=0 effort=-1 velocity=-1
- added joint Dummy_Platform: type fixed, parent Armar3_Base_link, child Dummy_Platform_link, origin xyz=0 0 0 rpy=-1.57079637 -0 0, axis 0 0 0, limit lower=0 upper=0 effort=-1 velocity=-1
- added joint Elbow L: type revolute, parent Upperarm L_link, child Elbow L_link, origin xyz=0.02 0 -0.31 rpy=-2.3561945 -1.57079625 -2.3561945, axis 0 0 1, limit lower=-1.5708 upper=0.331613 effort=-1 velocity=1
- added joint Elbow R: type revolute, parent Upperarm R_link, child Elbow R_link, origin xyz=0.02 0 -0.31 rpy=-2.3561945 -1.57079625 -2.3561945, axis 0 0 1, limit lower=-1.5708 upper=0.523599 effort=-1 velocity=1
- added joint EndArmL: type fixed, parent Wrist 2 L_link, child EndArmL_link, origin xyz=0 -0.04 0 rpy=1.57079637 -0 0, axis 0 0 0, limit lower=0 upper=0 effort=-1 velocity=-1
- added joint EndArmR: type fixed, parent Wrist 2 R_link, child EndArmR_link, origin xyz=0 -0.04 0 rpy=1.57079637 -0 0, axis 0 0 0, limit lower=0 upper=0 effort=-1 velocity=-1
- added joint EyeLeftCamera: type fixed, parent EyeLeftCameraPreTransformation_link, child EyeLeftCamera_link, origin xyz=0 0 0 rpy=0 -0 1.57079637, axis 0 0 0, limit lower=0 upper=0 effort=-1 velocity=-1
- added joint EyeLeftCameraPreTransformation: type fixed, parent Eye_Left_link, child EyeLeftCameraPreTransformation_link, origin xyz=0.02 0 0 rpy=3.14159274 1.57079625 3.14159274, axis 0 0 0, limit lower=0 upper=0 effort=-1 velocity=-1
- added joint EyeLeftCameraSim: type fixed, parent EyeLeftCameraPreTransformation_link, child EyeLeftCameraSim_link, origin xyz=0 0 0 rpy=0 -0 -3.1415925, axis 0 0 0, limit lower=0 upper=0 effort=-1 velocity=-1
- added joint EyeRightCamera: type fixed, parent EyeRightCameraPreTransformation_link, child EyeRightCamera_link, origin xyz=0 0 0 rpy=0 -0 1.57079637, axis 0 0 0, limit lower=0 upper=0 effort=-1 velocity=-1
- added joint EyeRightCameraPreTransformation: type fixed, parent Eye_Right_link, child EyeRightCameraPreTransformation_link, origin xyz=0.02 0 0 rpy=3.14159274 1.57079625 3.14159274, axis 0 0 0, limit lower=0 upper=0 effort=-1 velocity=-1
- added joint EyeRightCameraSim: type fixed, parent EyeRightCameraPreTransformation_link, child EyeRightCameraSim_link, origin xyz=0 0 0 rpy=0 -0 -3.1415925, axis 0 0 0, limit lower=0 upper=0 effort=-1 velocity=-1
- added joint Eye_Left: type revolute, parent Eye_Left_Dummy_link, child Eye_Left_link, origin xyz=0 0 0 rpy=0 -0 0, axis 0 0 1, limit lower=-0.523599 upper=0.523599 effort=-1 velocity=1
- added joint Eye_Left_Dummy: type fixed, parent Cameras_link, child Eye_Left_Dummy_link, origin xyz=0 0 0.0465 rpy=-1.57079637 -0 0, axis 0 0 0, limit lower=0 upper=0 effort=-1 velocity=-1
- added joint Eye_Right: type revolute, parent Eye_Right_Dummy_link, child Eye_Right_link, origin xyz=0 0 0 rpy=0 -0 0, axis 0 0 1, limit lower=-0.523599 upper=0.523599 effort=-1 velocity=1
- added joint Eye_Right_Dummy: type fixed, parent Cameras_link, child Eye_Right_Dummy_link, origin xyz=0 0 -0.0465 rpy=-1.57079637 -0 0, axis 0 0 0, limit lower=0 upper=0 effort=-1 velocity=-1
- added joint GCP L: type fixed, parent Hand L Base_link, child GCP L_link, origin xyz=-0.04 -0.02 0.09 rpy=0 -0.785398185 0, axis 0 0 0, limit lower=0 upper=0 effort=-1 velocity=-1
- added joint GCP R: type fixed, parent Hand R Base_link, child GCP R_link, origin xyz=-0.04 0.02 0.09 rpy=0 -0.785398185 0, axis 0 0 0, limit lower=0 upper=0 effort=-1 velocity=-1
- added joint Hand L Base: type fixed, parent EndArmL_link, child Hand L Base_link, origin xyz=0 0 0 rpy=0 -0 0, axis 0 0 0, limit lower=0 upper=0 effort=-1 velocity=-1
- added joint Hand Palm 1 L: type fixed, parent Hand L Base_link, child Hand Palm 1 L_link, origin xyz=0 0 0.036 rpy=0 -0 0, axis 0 0 0, limit lower=0 upper=0 effort=-1 velocity=-1
- added joint Hand Palm 1 R: type fixed, parent Hand R Base_link, child Hand Palm 1 R_link, origin xyz=0 0 0.036 rpy=0 -0 0, axis 0 0 0, limit lower=0 upper=0 effort=-1 velocity=-1
- added joint Hand Palm 2 L: type revolute, parent Hand Palm 1 L_link, child Hand Palm 2 L_link, origin xyz=-0.0087 0.0135 0.02925 rpy=0 -0 0, axis 0 -1 0, limit lower=-1.5708 upper=1.5708 effort=-1 velocity=1
- added joint Hand Palm 2 R: type revolute, parent Hand Palm 1 R_link, child Hand Palm 2 R_link, origin xyz=-0.0087 -0.0135 0.02925 rpy=0 -0 0, axis 0 -1 0, limit lower=-1.5708 upper=1.5708 effort=-1 velocity=1
- added joint Hand R Base: type fixed, parent EndArmR_link, child Hand R Base_link, origin xyz=0 0 0 rpy=0 -0 0, axis 0 0 0, limit lower=0 upper=0 effort=-1 velocity=-1
- added joint Head Base: type fixed, parent TrafoToHead_link, child Head Base_link, origin xyz=0 0 0 rpy=0 -0 1.57079637, axis 0 0 0, limit lower=0 upper=0 effort=-1 velocity=-1
- added joint Head Center: type fixed, parent Head Center1_link, child Head Center_link, origin xyz=0 0 0.0545 rpy=-1.57079637 -0 0, axis 0 0 0, limit lower=0 upper=0 effort=-1 velocity=-1
- added joint Head Center1: type fixed, parent Head_Tilt_link, child Head Center1_link, origin xyz=0 0 0 rpy=-1.57079637 -0 0, axis 0 0 0, limit lower=0 upper=0 effort=-1 velocity=-1
- added joint HeadIMU: type fixed, parent Head Center_link, child HeadIMU_link, origin xyz=0 -0.01 0 rpy=1.57079637 -0 0, axis 0 0 0, limit lower=0 upper=0 effort=-1 velocity=-1
- added joint HeadMotionMeasurementTCP: type fixed, parent EyeLeftCamera_link, child HeadMotionMeasurementTCP_link, origin xyz=0 0 1 rpy=0 -0 0, axis 0 0 0, limit lower=0 upper=0 effort=-1 velocity=-1
- added joint Head_Tilt: type revolute, parent Neck_3_Yaw_link, child Head_Tilt_link, origin xyz=0 0 0.12 rpy=1.57079637 -0 0, axis 0 0 1, limit lower=0 upper=0 effort=-1 velocity=1
- added joint Hip Pitch: type revolute, parent Platform_link, child Hip Pitch_link, origin xyz=0 0.158 0.89 rpy=0 -0 0, axis 1 0 0, limit lower=-0.785398 upper=0.785398 effort=-1 velocity=1
- added joint Hip Roll: type revolute, parent Hip Pitch_link, child Hip Roll_link, origin xyz=0 0 0 rpy=0 -0 0, axis 0 1 0, limit lower=-0.785398 upper=0.785398 effort=-1 velocity=1
- added joint Hip Yaw: type revolute, parent Hip Roll_link, child Hip Yaw_link, origin xyz=0 0 0 rpy=0 -0 0, axis 0 0 1, limit lower=-2.26893 upper=2.26893 effort=-1 velocity=1
- added joint Index L: type fixed, parent Hand Palm 2 L_link, child Index L_link, origin xyz=0 0 0.0402 rpy=0 -0 0, axis 0 0 0, limit lower=0 upper=0 effort=-1 velocity=-1
- added joint Index L J0: type revolute, parent Index L_link, child Index L J0_link, origin xyz=0 0 0 rpy=0 -0 0, axis 0 -1 0, limit lower=0 upper=3.14159 effort=-1 velocity=1
- added joint Index L J1: type revolute, parent Index L J0_link, child Index L J1_link, origin xyz=0 0 0.0402 rpy=0 -0 0, axis 0 -1 0, limit lower=0 upper=3.14159 effort=-1 velocity=1
- added joint Index R: type fixed, parent Hand Palm 2 R_link, child Index R_link, origin xyz=0 0 0.0402 rpy=0 -0 0, axis 0 0 0, limit lower=0 upper=0 effort=-1 velocity=-1
- added joint Index R Fingertip: type fixed, parent Index R J1_link, child Index R Fingertip_link, origin xyz=-0.005 0 0.0402 rpy=0 -0 0, axis 0 0 0, limit lower=0 upper=0 effort=-1 velocity=-1
- added joint Index R J0: type revolute, parent Index R_link, child Index R J0_link, origin xyz=0 0 0 rpy=0 -0 0, axis 0 -1 0, limit lower=0 upper=1.5708 effort=-1 velocity=1
- added joint Index R J1: type revolute, parent Index R J0_link, child Index R J1_link, origin xyz=0 0 0.0402 rpy=0 -0 0, axis 0 -1 0, limit lower=0 upper=1.5708 effort=-1 velocity=1
- added joint Jaw: type revolute, parent Head Center_link, child Jaw_link, origin xyz=0 0 0 rpy=0 -0 0, axis 0 0 1, limit lower=-0.523599 upper=0.523599 effort=-1 velocity=1
- added joint Kinect: type fixed, parent Head Center_link, child Kinect_link, origin xyz=0.14 -0.1 0 rpy=0 -0 0, axis 0 0 0, limit lower=0 upper=10000 effort=-1 velocity=1
- added joint Left Arm Base: type fixed, parent TrafoToLeftArm_link, child Left Arm Base_link, origin xyz=0 0 0 rpy=1.57079637 -0 -1.57079637, axis 0 0 0, limit lower=0 upper=0 effort=-1 velocity=-1
- added joint Lid Left Bottom: type revolute, parent Eye_Left_link, child Lid Left Bottom_link, origin xyz=0 0 0 rpy=0 -0 0, axis 0 1 0, limit lower=-3.14159 upper=3.14159 effort=-1 velocity=1
- added joint Lid Left Top: type revolute, parent Eye_Left_link, child Lid Left Top_link, origin xyz=0 0 0 rpy=0 -0 0, axis 0 1 0, limit lower=-3.14159 upper=3.14159 effort=-1 velocity=-1
- added joint Lid Right Bottom: type revolute, parent Eye_Right_link, child Lid Right Bottom_link, origin xyz=0 0 0 rpy=0 -0 0, axis 0 1 0, limit lower=-3.14159 upper=3.14159 effort=-1 velocity=1
- added joint Lid Right Top: type revolute, parent Eye_Right_link, child Lid Right Top_link, origin xyz=0 0 0 rpy=0 -0 0, axis 0 1 0, limit lower=-3.14159 upper=3.14159 effort=-1 velocity=1
- added joint Marker L: type fixed, parent Hand L Base_link, child Marker L_link, origin xyz=-0.035 0.045 0.065 rpy=0 -0 0, axis 0 0 0, limit lower=0 upper=0 effort=-1 velocity=-1
- added joint Marker R: type fixed, parent Hand R Base_link, child Marker R_link, origin xyz=-0.035 -0.045 0.065 rpy=0 -0 0, axis 0 0 0, limit lower=0 upper=0 effort=-1 velocity=-1
- added joint Middle L: type fixed, parent Hand Palm 2 L_link, child Middle L_link, origin xyz=0 -0.027 0.0404 rpy=0 -0 0, axis 0 0 0, limit lower=0 upper=0 effort=-1 velocity=-1
- added joint Middle L J0: type revolute, parent Middle L_link, child Middle L J0_link, origin xyz=0 0 0 rpy=0 -0 0, axis 0 -1 0, limit lower=0 upper=3.14159 effort=-1 velocity=1
- added joint Middle L J1: type revolute, parent Middle L J0_link, child Middle L J1_link, origin xyz=0 0 0.0402 rpy=0 -0 0, axis 0 -1 0, limit lower=0 upper=3.14159 effort=-1 velocity=1
- added joint Middle R: type fixed, parent Hand Palm 2 R_link, child Middle R_link, origin xyz=0 0.027 0.0404 rpy=0 -0 0, axis 0 0 0, limit lower=0 upper=0 effort=-1 velocity=-1
- added joint Middle R Fingertip: type fixed, parent Middle R J1_link, child Middle R Fingertip_link, origin xyz=-0.005 0 0.0402 rpy=0 -0 0, axis 0 0 0, limit lower=0 upper=0 effort=-1 velocity=-1
- added joint Middle R J0: type revolute, parent Middle R_link, child Middle R J0_link, origin xyz=0 0 0 rpy=0 -0 0, axis 0 -1 0, limit lower=0 upper=1.5708 effort=-1 velocity=1
- added joint Middle R J1: type revolute, parent Middle R J0_link, child Middle R J1_link, origin xyz=0 0 0.0402 rpy=0 -0 0, axis 0 -1 0, limit lower=0 upper=1.5708 effort=-1 velocity=1
- added joint Neck_1_Pitch: type revolute, parent Head Base_link, child Neck_1_Pitch_link, origin xyz=0 0 0 rpy=-2.3561945 -1.57079625 -2.3561945, axis 0 0 -1, limit lower=-0.785398 upper=0.645772 effort=-1 velocity=1
- added joint Neck_2_Roll: type revolute, parent Neck_1_Pitch_link, child Neck_2_Roll_link, origin xyz=0 0 0 rpy=-2.3561945 -1.57079625 -2.3561945, axis 0 0 1, limit lower=-0.785398 upper=0.785398 effort=-1 velocity=1
- added joint Neck_3_Yaw: type revolute, parent Neck_2_Roll_link, child Neck_3_Yaw_link, origin xyz=0 0 0 rpy=-2.3561945 -1.57079625 -2.3561945, axis 0 0 -1, limit lower=-2.0944 upper=2.0944 effort=-1 velocity=1
- added joint Pinky L: type fixed, parent Hand Palm 2 L_link, child Pinky L_link, origin xyz=0 -0.073 0.0404 rpy=0 -0 0, axis 0 0 0, limit lower=0 upper=0 effort=-1 velocity=-1
- added joint Pinky L J0: type revolute, parent Pinky L_link, child Pinky L J0_link, origin xyz=0 0 0 rpy=0 -0 0, axis 0 -1 0, limit lower=0 upper=3.14159 effort=-1 velocity=1
- added joint Pinky L J1: type revolute, parent Pinky L J0_link, child Pinky L J1_link, origin xyz=0 0 0.0402 rpy=0 -0 0, axis 0 -1 0, limit lower=0 upper=3.14159 effort=-1 velocity=1
- added joint Pinky R: type fixed, parent Hand Palm 2 R_link, child Pinky R_link, origin xyz=0 0.073 0.0404 rpy=0 -0 0, axis 0 0 0, limit lower=0 upper=0 effort=-1 velocity=-1
- added joint Pinky R J0: type revolute, parent Pinky R_link, child Pinky R J0_link, origin xyz=0 0 0 rpy=0 -0 0, axis 0 -1 0, limit lower=0 upper=1.5708 effort=-1 velocity=1
- added joint Pinky R J1: type revolute, parent Pinky R J0_link, child Pinky R J1_link, origin xyz=0 0 0.0402 rpy=0 -0 0, axis 0 -1 0, limit lower=0 upper=1.5708 effort=-1 velocity=1
- added joint Platform: type fixed, parent Yaw_Platform_link, child Platform_link, origin xyz=0 0 0 rpy=0 -0 0, axis 0 0 0, limit lower=0 upper=0 effort=-1 velocity=-1
- added joint Right Arm Base: type fixed, parent TrafoToRightArm_link, child Right Arm Base_link, origin xyz=0 0 0 rpy=1.57079637 -0 -1.57079637, axis 0 0 0, limit lower=0 upper=0 effort=-1 velocity=-1
- added joint Ring L: type fixed, parent Hand Palm 2 L_link, child Ring L_link, origin xyz=0 -0.051 0.0404 rpy=0 -0 0, axis 0 0 0, limit lower=0 upper=0 effort=-1 velocity=-1
- added joint Ring L J0: type revolute, parent Ring L_link, child Ring L J0_link, origin xyz=0 0 0 rpy=0 -0 0, axis 0 -1 0, limit lower=0 upper=3.14159 effort=-1 velocity=1
- added joint Ring L J1: type revolute, parent Ring L J0_link, child Ring L J1_link, origin xyz=0 0 0.0402 rpy=0 -0 0, axis 0 -1 0, limit lower=0 upper=3.14159 effort=-1 velocity=1
- added joint Ring R: type fixed, parent Hand Palm 2 R_link, child Ring R_link, origin xyz=0 0.051 0.0404 rpy=0 -0 0, axis 0 0 0, limit lower=0 upper=0 effort=-1 velocity=-1
- added joint Ring R J0: type revolute, parent Ring R_link, child Ring R J0_link, origin xyz=0 0 0 rpy=0 -0 0, axis 0 -1 0, limit lower=0 upper=1.5708 effort=-1 velocity=1
- added joint Ring R J1: type revolute, parent Ring R J0_link, child Ring R J1_link, origin xyz=0 0 0.0402 rpy=0 -0 0, axis 0 -1 0, limit lower=0 upper=1.5708 effort=-1 velocity=1
- added joint Shoulder 1 L: type revolute, parent Left Arm Base_link, child Shoulder 1 L_link, origin xyz=0 0 0 rpy=0 -0 1.57079637, axis 0 0 1, limit lower=-1.8675 upper=0.733038 effort=-1 velocity=1
- added joint Shoulder 1 R: type revolute, parent Right Arm Base_link, child Shoulder 1 R_link, origin xyz=0 0 0 rpy=0 -0 1.57079637, axis 0 0 1, limit lower=-1.8675 upper=0.733038 effort=-1 velocity=0.5
- added joint Shoulder 2 L: type revolute, parent Shoulder 1 L_link, child Shoulder 2 L_link, origin xyz=0 0 0 rpy=1.57079649 -1.30899692 -1.63133095e-07, axis 0 0 -1, limit lower=-0.244346 upper=1.65806 effort=-1 velocity=1
- added joint Shoulder 2 R: type revolute, parent Shoulder 1 R_link, child Shoulder 2 R_link, origin xyz=0 0 0 rpy=-1.57079649 -1.30899692 -3.1415925, axis 0 0 1, limit lower=-0.244346 upper=1.65806 effort=-1 velocity=0.5
- added joint TCP L: type fixed, parent Hand L Base_link, child TCP L_link, origin xyz=0 0 0.13 rpy=0 -0 0, axis 0 0 0, limit lower=0 upper=0 effort=-1 velocity=-1
- added joint TCP R: type fixed, parent Hand R Base_link, child TCP R_link, origin xyz=0 0 0.13 rpy=0 -0 0, axis 0 0 0, limit lower=0 upper=0 effort=-1 velocity=-1
- added joint Thumb L: type fixed, parent Hand Palm 1 L_link, child Thumb L_link, origin xyz=-0.0489 0 0.02925 rpy=0 -0 0, axis 0 0 0, limit lower=0 upper=0 effort=-1 velocity=-1
- added joint Thumb L J0: type revolute, parent Thumb L_link, child Thumb L J0_link, origin xyz=0 0 0 rpy=0 -0 0, axis 0 1 0, limit lower=0 upper=3.14159 effort=-1 velocity=1
- added joint Thumb L J1: type revolute, parent Thumb L J0_link, child Thumb L J1_link, origin xyz=-0.0402 0 0 rpy=0 -0 0, axis 0 1 0, limit lower=0 upper=3.14159 effort=-1 velocity=1
- added joint Thumb R: type fixed, parent Hand Palm 1 R_link, child Thumb R_link, origin xyz=-0.0489 0 0.02925 rpy=0 -0 0, axis 0 0 0, limit lower=0 upper=0 effort=-1 velocity=-1
- added joint Thumb R Fingertip: type fixed, parent Thumb R J1_link, child Thumb R Fingertip_link, origin xyz=-0.05 0 0 rpy=0 -0 0, axis 0 0 0, limit lower=0 upper=0 effort=-1 velocity=-1
- added joint Thumb R J0: type revolute, parent Thumb R_link, child Thumb R J0_link, origin xyz=0 0 0 rpy=0 -0 0, axis 0 1 0, limit lower=0 upper=1.5708 effort=-1 velocity=1
- added joint Thumb R J1: type revolute, parent Thumb R J0_link, child Thumb R J1_link, origin xyz=-0.0402 0 0 rpy=0 -0 0, axis 0 1 0, limit lower=0 upper=1.5708 effort=-1 velocity=1
- added joint TrafoToHead: type fixed, parent Center of Arms_link, child TrafoToHead_link, origin xyz=0 0 0.118 rpy=0 -0 0, axis 0 0 0, limit lower=0 upper=0 effort=-1 velocity=-1
- added joint TrafoToLeftArm: type fixed, parent Center of Arms_link, child TrafoToLeftArm_link, origin xyz=-0.232 0 0 rpy=0 -0 0, axis 0 0 0, limit lower=0 upper=0 effort=-1 velocity=-1
- added joint TrafoToRightArm: type fixed, parent Center of Arms_link, child TrafoToRightArm_link, origin xyz=0.232 0 0 rpy=0 -0 0, axis 0 0 0, limit lower=0 upper=0 effort=-1 velocity=-1
- added joint Underarm L: type revolute, parent Elbow L_link, child Underarm L_link, origin xyz=0 0 -0.0075 rpy=2.3561945 1.57079625 -2.3561945, axis 0 0 -1, limit lower=-1.5708 upper=2.75762 effort=-1 velocity=1
- added joint Underarm R: type revolute, parent Elbow R_link, child Underarm R_link, origin xyz=0 0 0.0075 rpy=2.3561945 1.57079625 -2.3561945, axis 0 0 1, limit lower=-1.5708 upper=3.49066 effort=-1 velocity=0.5
- added joint Upperarm L: type revolute, parent Shoulder 2 L_link, child Upperarm L_link, origin xyz=0 0 0 rpy=-2.3561945 1.57079625 2.3561945, axis 0 0 -1, limit lower=-1.22173 upper=1.22173 effort=-1 velocity=1
- added joint Upperarm R: type revolute, parent Shoulder 2 R_link, child Upperarm R_link, origin xyz=0 0 0 rpy=-2.3561945 1.57079625 2.3561945, axis 0 0 1, limit lower=-1.90241 upper=1.22173 effort=-1 velocity=0.5
- added joint VirtualCentralGaze: type fixed, parent Cameras_link, child VirtualCentralGaze_link, origin xyz=0 0 0 rpy=0 -0 0, axis 0 0 0, limit lower=0 upper=10000 effort=-1 velocity=1
- added joint Wrist 1 L: type revolute, parent Underarm L_link, child Wrist 1 L_link, origin xyz=0 0 -0.24 rpy=2.3561945 -1.57079625 2.3561945, axis 0 0 -1, limit lower=-0.506145 upper=0.523599 effort=-1 velocity=1
- added joint Wrist 1 R: type revolute, parent Underarm R_link, child Wrist 1 R_link, origin xyz=0 0 -0.24 rpy=2.3561945 -1.57079625 2.3561945, axis 0 0 1, limit lower=-0.389208 upper=0.397935 effort=-1 velocity=0.5
- added joint Wrist 2 L: type revolute, parent Wrist 1 L_link, child Wrist 2 L_link, origin xyz=0 0 0 rpy=2.3561945 -1.57079625 2.3561945, axis 0 0 1, limit lower=-0.663225 upper=0.767945 effort=-1 velocity=1
- added joint Wrist 2 R: type revolute, parent Wrist 1 R_link, child Wrist 2 R_link, origin xyz=0 0 0 rpy=2.3561945 -1.57079625 2.3561945, axis 0 0 1, limit lower=-0.541052 upper=0.645772 effort=-1 velocity=0.5
- added joint X_Platform: type prismatic, parent Dummy_Platform_link, child X_Platform_link, origin xyz=0 0 0 rpy=-1.57079637 -0 1.57079637, axis 0 0 -1, limit lower=-0 upper=5000 effort=-1 velocity=-1
- added joint Y_Platform: type prismatic, parent X_Platform_link, child Y_Platform_link, origin xyz=0 0 0 rpy=1.57079637 -0 -1.57079637, axis 1 0 0, limit lower=0 upper=10000 effort=-1 velocity=-1
- added joint Yaw_Platform: type revolute, parent Y_Platform_link, child Yaw_Platform_link, origin xyz=0 0 0 rpy=0 -0 -1.57079637, axis 0 0 1, limit lower=-6.28319 upper=6.28319 effort=-1 velocity=1
- added joint left_hand_configuration_actual_float: type fixed, parent Hand L Base_link, child left_hand_configuration_actual_float_link, origin xyz=0 0 0 rpy=0 -0 0, axis 0 0 0, limit lower=0 upper=0 effort=-1 velocity=-1
- added joint right_hand_configuration_actual_float: type fixed, parent Hand R Base_link, child right_hand_configuration_actual_float_link, origin xyz=0 0 0 rpy=0 -0 0, axis 0 0 0, limit lower=0 upper=0 effort=-1 velocity=-1
