Commit message: enable model export

File: data/robots/Armar3/urdf/Armar3.urdf (robot description, URDF)
Before this commit: robot Armar3, 108 links, 107 joints
Links:
- link Wrist 1 L_link: geometry collision mesh filename=stl/wrist1_l.stl scale=1 1 1; visual mesh filename=fullmodel/wrist1_l.iv scale=1 1 1
- link Wrist 1 R_link: geometry collision mesh filename=stl/wrist1_r.stl scale=1 1 1; visual mesh filename=fullmodel/wrist1_r.iv scale=1 1 1
- link Wrist 2 L_link: geometry visual mesh filename=fullmodel/wrist2_l.iv scale=1 1 1
- link Wrist 2 R_link: geometry visual mesh filename=fullmodel/wrist2_r.iv scale=1 1 1

Commit message: fixed warnings when loading armar3

File: data/robots/Armar3/urdf/Armar3.urdf (robot description, URDF)
Before this commit: robot Armar3, 108 links, 107 joints
Links:
- link Cameras_link: geometry 
- link Eye_Left_link: geometry visual mesh filename=fullmodel/eye_l.iv scale=1 1 1
- link Eye_Right_link: geometry visual mesh filename=fullmodel/eye_r.iv scale=1 1 1

Commit message: Add collada version of Armar3

File: data/robots/Armar3/urdf/Armar3.urdf (robot description, URDF)
Before this commit: robot Armar3, 108 links, 107 joints
Links:
- link Elbow L_link: geometry collision mesh filename=stl/elbow_l.stl scale=1000 1000 1000; visual mesh filename=fullmodel/elbow_l.dae scale=1000 1000 1000
- link Elbow R_link: geometry collision mesh filename=stl/elbow_r.stl scale=1000 1000 1000; visual mesh filename=fullmodel/elbow_r.dae scale=1000 1000 1000
- link Eye_Left_link: geometry visual mesh filename=fullmodel/eye_l.dae scale=1000 1000 1000
- link Eye_Right_link: geometry visual mesh filename=fullmodel/eye_r.dae scale=1000 1000 1000
- link Hand Palm 1 L_link: geometry collision mesh filename=stl/palm1_l.stl scale=1000 1000 1000; visual mesh filename=fullmodel/palm1_l.dae scale=1000 1000 1000
- link Hand Palm 1 R_link: geometry collision mesh filename=stl/palm1_r.stl scale=1000 1000 1000; visual mesh filename=fullmodel/palm1_r.dae scale=1000 1000 1000
- link Hand Palm 2 L_link: geometry collision mesh filename=stl/palm2_l.stl scale=1000 1000 1000; visual mesh filename=fullmodel/palm2_l.dae scale=1000 1000 1000
- link Hand Palm 2 R_link: geometry collision mesh filename=stl/palm2_r.stl scale=1000 1000 1000; visual mesh filename=fullmodel/palm2_r.dae scale=1000 1000 1000
- link Head Base_link: geometry collision mesh filename=stl/head_base.stl scale=1000 1000 1000; visual mesh filename=fullmodel/head_base.dae scale=1000 1000 1000
- link Head_Tilt_link: geometry collision mesh filename=stl/head.stl scale=1000 1000 1000; visual mesh filename=fullmodel/head.dae scale=1000 1000 1000
- link Hip Pitch_link: geometry collision mesh filename=stl/platform_pitch_link.stl scale=1000 1000 1000; visual mesh filename=fullmodel/platform_pitch_link.dae scale=1000 1000 1000
- link Hip Roll_link: geometry collision mesh filename=stl/platform_roll_link.stl scale=1000 1000 1000; visual mesh filename=fullmodel/platform_roll_link.dae scale=1000 1000 1000
- link Hip Yaw_link: geometry collision mesh filename=stl/torso.stl scale=1000 1000 1000; visual mesh filename=fullmodel/torso.dae scale=1000 1000 1000
- link Index L J0_link: geometry collision mesh filename=stl/index_l1.stl scale=1000 1000 1000; visual mesh filename=fullmodel/index_l1.dae scale=1000 1000 1000
- link Index L J1_link: geometry collision mesh filename=stl/index_l2.stl scale=1000 1000 1000; visual mesh filename=fullmodel/index_l2.dae scale=1000 1000 1000
- link Index R J0_link: geometry collision mesh filename=stl/index_r1.stl scale=1000 1000 1000; visual mesh filename=fullmodel/index_r1.dae scale=1000 1000 1000
- link Index R J1_link: geometry collision mesh filename=stl/index_r2.stl scale=1000 1000 1000; visual mesh filename=fullmodel/index_r2.dae scale=1000 1000 1000
- link Jaw_link: geometry visual mesh filename=fullmodel/jaw.dae scale=1000 1000 1000
- link Lid Left Bottom_link: geometry visual mesh filename=fullmodel/lid_l_bottom.dae scale=1000 1000 1000
- link Lid Left Top_link: geometry visual mesh filename=fullmodel/lid_l_top.dae scale=1000 1000 1000
- link Lid Right Bottom_link: geometry visual mesh filename=fullmodel/lid_r_bottom.dae scale=1000 1000 1000
- link Lid Right Top_link: geometry visual mesh filename=fullmodel/lid_r_top.dae scale=1000 1000 1000
- link Middle L J0_link: geometry collision mesh filename=stl/middle_l1.stl scale=1000 1000 1000; visual mesh filename=fullmodel/middle_l1.dae scale=1000 1000 1000
- link Middle L J1_link: geometry collision mesh filename=stl/middle_l2.stl scale=1000 1000 1000; visual mesh filename=fullmodel/middle_l2.dae scale=1000 1000 1000
- link Middle R J0_link: geometry collision mesh filename=stl/middle_r1.stl scale=1000 1000 1000; visual mesh filename=fullmodel/middle_r1.dae scale=1000 1000 1000
- link Middle R J1_link: geometry collision mesh filename=stl/middle_r2.stl scale=1000 1000 1000; visual mesh filename=fullmodel/middle_r2.dae scale=1000 1000 1000
- link Neck_1_Pitch_link: geometry collision mesh filename=stl/neck_pitch_link.stl scale=1000 1000 1000; visual mesh filename=fullmodel/neck_pitch_link.dae scale=1000 1000 1000
- link Neck_2_Roll_link: geometry collision mesh filename=stl/neck_roll_link.stl scale=1000 1000 1000; visual mesh filename=fullmodel/neck_roll_link.dae scale=1000 1000 1000
- link Neck_3_Yaw_link: geometry collision mesh filename=stl/neck_yaw_link.stl scale=1000 1000 1000; visual mesh filename=fullmodel/neck_yaw_link.dae scale=1000 1000 1000
- link Pinky L J0_link: geometry collision mesh filename=stl/pinky_l1.stl scale=1000 1000 1000; visual mesh filename=fullmodel/pinky_l1.dae scale=1000 1000 1000
- link Pinky L J1_link: geometry collision mesh filename=stl/pinky_l2.stl scale=1000 1000 1000; visual mesh filename=fullmodel/pinky_l2.dae scale=1000 1000 1000
- link Pinky R J0_link: geometry collision mesh filename=stl/pinky_r1.stl scale=1000 1000 1000; visual mesh filename=fullmodel/pinky_r1.dae scale=1000 1000 1000
- link Pinky R J1_link: geometry collision mesh filename=stl/pinky_r2.stl scale=1000 1000 1000; visual mesh filename=fullmodel/pinky_r2.dae scale=1000 1000 1000
- link Platform_link: geometry collision mesh filename=stl/platform.stl scale=1000 1000 1000; visual mesh filename=fullmodel/platform.dae scale=1000 1000 1000
- link Ring L J0_link: geometry collision mesh filename=stl/ring_l1.stl scale=1000 1000 1000; visual mesh filename=fullmodel/ring_l1.dae scale=1000 1000 1000
- link Ring L J1_link: geometry collision mesh filename=stl/ring_l2.stl scale=1000 1000 1000; visual mesh filename=fullmodel/ring_l2.dae scale=1000 1000 1000
- link Ring R J0_link: geometry collision mesh filename=stl/ring_r1.stl scale=1000 1000 1000; visual mesh filename=fullmodel/ring_r1.dae scale=1000 1000 1000
- link Ring R J1_link: geometry collision mesh filename=stl/ring_r2.stl scale=1000 1000 1000; visual mesh filename=fullmodel/ring_r2.dae scale=1000 1000 1000
- link Shoulder 1 L_link: geometry collision mesh filename=stl/shoulder_l.stl scale=1000 1000 1000; visual mesh filename=fullmodel/shoulder_l.dae scale=1000 1000 1000
- link Shoulder 1 R_link: geometry collision mesh filename=stl/shoulder_r.stl scale=1000 1000 1000; visual mesh filename=fullmodel/shoulder_r.dae scale=1000 1000 1000
- link Shoulder 2 L_link: geometry collision mesh filename=stl/shoulder2_l_rot.stl scale=1000 1000 1000; visual mesh filename=fullmodel/shoulder2_l_rot.dae scale=1000 1000 1000
- link Shoulder 2 R_link: geometry collision mesh filename=stl/shoulder2_r_rot.stl scale=1000 1000 1000; visual mesh filename=fullmodel/shoulder2_r_rot.dae scale=1000 1000 1000
- link Thumb L J0_link: geometry collision mesh filename=stl/thumb_l1.stl scale=1000 1000 1000; visual mesh filename=fullmodel/thumb_l1.dae scale=1000 1000 1000
- link Thumb L J1_link: geometry collision mesh filename=stl/thumb_l2.stl scale=1000 1000 1000; visual mesh filename=fullmodel/thumb_l2.dae scale=1000 1000 1000
- link Thumb R J0_link: geometry collision mesh filename=stl/thumb_r1.stl scale=1000 1000 1000; visual mesh filename=fullmodel/thumb_r1.dae scale=1000 1000 1000
- link Thumb R J1_link: geometry collision mesh filename=stl/thumb_r2.stl scale=1000 1000 1000; visual mesh filename=fullmodel/thumb_r2.dae scale=1000 1000 1000
- link Underarm L_link: geometry collision mesh filename=stl/underarm_l.stl scale=1000 1000 1000; visual mesh filename=fullmodel/underarm_l.dae scale=1000 1000 1000
- link Underarm R_link: geometry collision mesh filename=stl/underarm_r.stl scale=1000 1000 1000; visual mesh filename=fullmodel/underarm_r.dae scale=1000 1000 1000
- link Upperarm L_link: geometry collision mesh filename=stl/upperarm_l.stl scale=1000 1000 1000; visual mesh filename=fullmodel/upperarm_l.dae scale=1000 1000 1000
- link Upperarm R_link: geometry collision mesh filename=stl/upperarm_r.stl scale=1000 1000 1000; visual mesh filename=fullmodel/upperarm_r.dae scale=1000 1000 1000
- link Wrist 1 L_link: geometry collision mesh filename=stl/wrist1_l.stl scale=1000 1000 1000; visual mesh filename=fullmodel/wrist1_l.dae scale=1000 1000 1000
- link Wrist 1 R_link: geometry collision mesh filename=stl/wrist1_r.stl scale=1000 1000 1000; visual mesh filename=fullmodel/wrist1_r.dae scale=1000 1000 1000
- link Wrist 2 L_link: geometry visual mesh filename=fullmodel/wrist2_l.dae scale=1000 1000 1000
- link Wrist 2 R_link: geometry visual mesh filename=fullmodel/wrist2_r.dae scale=1000 1000 1000
