Commit message: update point grasp position

File: VirtualRobot/data/robots/urdf/Pepper/urdf/pepper_LGripper.urdf (robot description, URDF)
Before this commit: robot LGripper, 19 links, 18 joints
Joints:
- joint LGripperEef: origin xyz=0.025 0 -0.030 rpy=3.14 -0.785 0 -> xyz=0.020 0 -0.005 rpy=3.14 -0.785 0

File: VirtualRobot/data/robots/urdf/Pepper/urdf/pepper_RGripper.urdf (robot description, URDF)
Before this commit: robot RGripper, 19 links, 18 joints
Joints:
- joint RGripperEef: origin xyz=0.025 0 -0.030 rpy=3.14 -0.785 0 -> xyz=0.020 0 -0.005 rpy=3.14 -0.785 0

Commit message: update hand description with new R/LGripper

File: VirtualRobot/data/robots/urdf/Pepper/urdf/pepper_LGripper.urdf (robot description, URDF)
Before this commit: robot LGripper, 19 links, 18 joints
Links:
- removed link l_eef
- added link l_hand, mass 2e-03
Joints:
- removed joint LGripperEef
- added joint LGripper: type fixed, parent l_wrist, child l_gripper, origin xyz=0.07 0.0 -0.01802319018 rpy=-3.14 0.0 -1.57, axis 0 0 0
- joint LHand: child l_gripper -> l_hand

File: VirtualRobot/data/robots/urdf/Pepper/urdf/pepper_RGripper.urdf (robot description, URDF)
Before this commit: robot RGripper, 19 links, 18 joints
Links:
- removed link r_eef
- added link r_hand, mass 2e-03
Joints:
- removed joint RGripperEef
- added joint RGripper: type fixed, parent r_wrist, child r_gripper, origin xyz=0.07 0.0 -0.01802319018 rpy=3.14 0 1.57, axis 0 0 0
- joint RHand: child r_gripper -> r_hand
